Commit message: format of URDF files

File: jaco_model/urdf/jaco_arm_back.xacro (robot description, xacro)
@@ -2,131 +2,129 @@
 <root xmlns:xi="http://www.w3.org/2001/XInclude"
 	xmlns:gazebo="http://playerstage.sourceforge.net/gazebo/xmlschema/#gz"
-    xmlns:model="http://playerstage.sourceforge.net/gazebo/xmlschema/#model"
+	xmlns:model="http://playerstage.sourceforge.net/gazebo/xmlschema/#model"
 	xmlns:sensor="http://playerstage.sourceforge.net/gazebo/xmlschema/#sensor"
 	xmlns:body="http://playerstage.sourceforge.net/gazebo/xmlschema/#body"
-    xmlns:geom="http://playerstage.sourceforge.net/gazebo/xmlschema/#geom"
-    xmlns:joint="http://playerstage.sourceforge.net/gazebo/xmlschema/#joint"
+	xmlns:geom="http://playerstage.sourceforge.net/gazebo/xmlschema/#geom"
+	xmlns:joint="http://playerstage.sourceforge.net/gazebo/xmlschema/#joint"
 	xmlns:controller="http://playerstage.sourceforge.net/gazebo/xmlschema/#controller"
 	xmlns:interface="http://playerstage.sourceforge.net/gazebo/xmlschema/#interface"
 	xmlns:rendering="http://playerstage.sourceforge.net/gazebo/xmlschema/#rendering"
-    xmlns:renderable="http://playerstage.sourceforge.net/gazebo/xmlschema/#renderable"
-    xmlns:physics="http://playerstage.sourceforge.net/gazebo/xmlschema/#physics"
+	xmlns:renderable="http://playerstage.sourceforge.net/gazebo/xmlschema/#renderable"
+	xmlns:physics="http://playerstage.sourceforge.net/gazebo/xmlschema/#physics"
 	xmlns:xacro="http://ros.org/wiki/xacro">
-  <property name="J_PI" value="3.1415926535897931" />
-  <property name="J_LIM" value="${2*J_PI}" />
-  <property name="link_base" value="jaco_link_base" />
-  <property name="link_1" value="jaco_link_1" />
-  <property name="link_2" value="jaco_link_2" />
-  <property name="link_3" value="jaco_link_3" />
-  <property name="link_4" value="jaco_link_4" />
-  <property name="link_5" value="jaco_link_5" />
-  <property name="link_hand" value="jaco_link_hand" />
-  <property name="link_finger_1" value="jaco_link_finger_1" />
-  <property name="link_finger_2" value="jaco_link_finger_2" />
-  <property name="link_finger_3" value="jaco_link_finger_3" />
-  <property name="joint_base" value="jaco_joint_base" />
-  <property name="joint_base_axis_xyz" value="0 0 0" />
-  <property name="joint_base_origin_xyz" value="0 0 0" />
-  <property name="joint_base_origin_rpy" value="0 0 0" />
-  <property name="joint_1" value="jaco_joint_1" />
-  <property name="joint_1_axis_xyz" value="0 0 1" />
-  <property name="joint_1_origin_xyz" value="0 0 0.1535" />
-  <property name="joint_1_origin_rpy" value="${J_PI} 0 0" />
-  <property name="joint_2" value="jaco_joint_2" />
-  <property name="joint_2_axis_xyz" value="0 0 1" />
-  <property name="joint_2_origin_xyz" value="0 0 -0.1185" />
-  <property name="joint_2_origin_rpy" value="-${J_PI/2} -${J_PI/2} 0" />
-  <property name="joint_3" value="jaco_joint_3" />
-  <property name="joint_3_axis_xyz" value="0 0 1" />
-  <property name="joint_3_origin_xyz" value="0.41 0 0" />
-  <property name="joint_3_origin_rpy" value="${J_PI} 0 ${J_PI}" />
-  <property name="joint_4" value="jaco_joint_4" />
-  <property name="joint_4_axis_xyz" value="0 0 1" />
-  <property name="joint_4_origin_xyz" value="0.207 0 -0.01125" />
-  <property name="joint_4_origin_rpy" value="0 -${J_PI/2} 0" />
-  <property name="joint_5" value="jaco_joint_5" />
-  <property name="joint_5_axis_xyz" value="0 0 1" />
-  <property name="joint_5_origin_xyz" value="0.0343 0 -0.06588" />
-  <property name="joint_5_origin_rpy" value="0 ${J_PI/180*55} ${J_PI}" />
-  <property name="joint_6" value="jaco_joint_6" />
-  <property name="joint_6_axis_xyz" value="0 0 1" />
-  <property name="joint_6_origin_xyz" value="0.0343 0 -0.06588" />
-  <property name="joint_6_origin_rpy" value="0 ${J_PI/180*55} ${J_PI}" />
-  <property name="joint_finger_1" value="jaco_joint_finger_1" />
-  <property name="joint_finger_1_axis_xyz" value="0 0 1" />
-  <property name="joint_finger_1_origin_xyz" value="-0.03978 0 -0.10071" />
-  <property name="joint_finger_1_origin_rpy" value="-1.7983 1.117 3.1416" />
-  <property name="joint_finger_1_lower_limit" value="0" />
-  <property name="joint_finger_1_upper_limit" value="${J_PI/180*40}" />
-  <property name="joint_finger_2" value="jaco_joint_finger_2" />
-  <property name="joint_finger_2_axis_xyz" value="0 0 1" />
-  <property name="joint_finger_2_origin_xyz" value="0.03569 -0.0216 -0.10071" />
-  <property name="joint_finger_2_origin_rpy" value="-1.6222 1.117 -0.23615" />
-  <property name="joint_finger_2_lower_limit" value="0" />
-  <property name="joint_finger_2_upper_limit" value="${J_PI/180*40}" />
-  <property name="joint_finger_3" value="jaco_joint_finger_3" />
-  <property name="joint_finger_3_axis_xyz" value="0 0 1" />
-  <property name="joint_finger_3_origin_xyz" value="0.03569 0.0216 -0.10071" />
-  <property name="joint_finger_3_origin_rpy" value="-1.5161 1.1459 0.23978" />
-  <property name="joint_finger_3_lower_limit" value="0" />
-  <property name="joint_finger_3_upper_limit" value="${J_PI/180*40}" />
-<xacro:macro name="jaco_link" params="link_name">
-<link name="${link_name}">
-      <visual>
-                 <geometry>
-                         <mesh
-          filename="package://jaco_model/meshes/${link_name}.dae"/>
-                </geometry>
-                <material name="carbon_fiber">
- 			<color rgba="0.792156862745098 0.819607843137255 0.933333333333333 1" />
-                </material>
-        </visual>
-        <collision>
-                <geometry>
-                         <mesh
-          filename="package://jaco_model/meshes/${link_name}.dae"/>
-                </geometry>
-        </collision>
-</link>
-</xacro:macro>
-<xacro:macro name="jaco_joint" params="joint_name type parent child joint_axis_xyz joint_origin_xyz joint_origin_rpy lower_limit upper_limit">
-<joint name="${joint_name}" type="${type}">
-    <parent link="${parent}"/>
-    <child link="${child}"/>
-    <axis xyz="${joint_axis_xyz}"/>
-<origin xyz="${joint_origin_xyz}" rpy="${joint_origin_rpy}"/>
- <limit lower="${lower_limit}" upper="${upper_limit}" effort="30" velocity="5"/>
- </joint>
-</xacro:macro>
-<xacro:macro name="jaco_finger_joint" params="joint_name type parent child joint_axis_xyz joint_origin_xyz joint_origin_rpy lower_limit upper_limit">
-<joint name="${joint_name}" type="${type}">
-    <parent link="${parent}"/>
-    <child link="${child}"/>
-    <axis xyz="${joint_axis_xyz}"/>
-<origin xyz="${joint_origin_xyz}" rpy="${joint_origin_rpy}"/>
-    <limit lower="${lower_limit}" upper="${upper_limit}" effort="30" velocity="5"/>
- </joint>
-</xacro:macro>
-<xacro:macro name="jaco_arm" params="parent">
-   <xacro:jaco_link link_name="${link_base}"/>
-   <xacro:jaco_joint joint_name="${joint_base}" type="fixed" parent="${parent}" child="${link_base}" joint_axis_xyz="${joint_base_axis_xyz}" joint_origin_xyz="${joint_base_origin_xyz}" joint_origin_rpy="${joint_base_origin_rpy}" lower_limit="-${J_LIM}" upper_limit="${J_LIM}"/>
-   <xacro:jaco_link link_name="${link_1}"/>
-   <xacro:jaco_joint joint_name="${joint_1}" type="revolute" parent="${link_base}" child="${link_1}" joint_axis_xyz="${joint_1_axis_xyz}" joint_origin_xyz="${joint_1_origin_xyz}" joint_origin_rpy="${joint_1_origin_rpy}" lower_limit="-${J_LIM}" upper_limit="${J_LIM}"/>
-   <xacro:jaco_link link_name="${link_2}"/>
-   <xacro:jaco_joint joint_name="${joint_2}" type="revolute" parent="${link_1}" child="${link_2}" joint_axis_xyz="${joint_2_axis_xyz}" joint_origin_xyz="${joint_2_origin_xyz}" joint_origin_rpy="${joint_2_origin_rpy}" lower_limit="0" upper_limit="${J_LIM}"/>
-   <xacro:jaco_link link_name="${link_3}"/>
-   <xacro:jaco_joint joint_name="${joint_3}" type="revolute" parent="${link_2}" child="${link_3}" joint_axis_xyz="${joint_3_axis_xyz}" joint_origin_xyz="${joint_3_origin_xyz}" joint_origin_rpy="${joint_3_origin_rpy}" lower_limit="0" upper_limit="${J_LIM}"/>
-   <xacro:jaco_link link_name="${link_4}"/>
-   <xacro:jaco_joint joint_name="${joint_4}" type="revolute" parent="${link_3}" child="${link_4}" joint_axis_xyz="${joint_4_axis_xyz}" joint_origin_xyz="${joint_4_origin_xyz}" joint_origin_rpy="${joint_4_origin_rpy}" lower_limit="-${J_LIM}" upper_limit="${J_LIM}"/>
-   <xacro:jaco_link link_name="${link_5}"/>
-   <xacro:jaco_joint joint_name="${joint_5}" type="revolute" parent="${link_4}" child="${link_5}" joint_axis_xyz="${joint_5_axis_xyz}" joint_origin_xyz="${joint_5_origin_xyz}" joint_origin_rpy="${joint_5_origin_rpy}" lower_limit="-${J_LIM}" upper_limit="${J_LIM}"/>
-   <xacro:jaco_link link_name="${link_hand}"/>
-   <xacro:jaco_joint joint_name="${joint_6}" type="revolute" parent="${link_5}" child="${link_hand}" joint_axis_xyz="${joint_6_axis_xyz}" joint_origin_xyz="${joint_6_origin_xyz}" joint_origin_rpy="${joint_6_origin_rpy}" lower_limit="-${J_LIM}" upper_limit="${J_LIM}"/>
-   <xacro:jaco_link link_name="${link_finger_1}"/>
-   <xacro:jaco_finger_joint joint_name="${joint_finger_1}" type="revolute" parent="${link_hand}" child="${link_finger_1}" joint_axis_xyz="${joint_finger_1_axis_xyz}" joint_origin_xyz="${joint_finger_1_origin_xyz}" joint_origin_rpy="${joint_finger_1_origin_rpy}" lower_limit="${joint_finger_1_lower_limit}" upper_limit="${joint_finger_1_upper_limit}"/>
-   <xacro:jaco_link link_name="${link_finger_2}"/>
-   <xacro:jaco_finger_joint joint_name="${joint_finger_2}" type="revolute" parent="${link_hand}" child="${link_finger_2}" joint_axis_xyz="${joint_finger_2_axis_xyz}" joint_origin_xyz="${joint_finger_2_origin_xyz}" joint_origin_rpy="${joint_finger_2_origin_rpy}" lower_limit="${joint_finger_2_lower_limit}" upper_limit="${joint_finger_2_upper_limit}"/>
-   <xacro:jaco_link link_name="${link_finger_3}"/>
-   <xacro:jaco_finger_joint joint_name="${joint_finger_3}" type="revolute" parent="${link_hand}" child="${link_finger_3}" joint_axis_xyz="${joint_finger_3_axis_xyz}" joint_origin_xyz="${joint_finger_3_origin_xyz}" joint_origin_rpy="${joint_finger_3_origin_rpy}" lower_limit="${joint_finger_3_lower_limit}" upper_limit="${joint_finger_3_upper_limit}"/>
-</xacro:macro>
+	<property name="J_PI" value="3.1415926535897931" />
+	<property name="J_LIM" value="${2*J_PI}" />
+	<property name="link_base" value="jaco_link_base" />
+	<property name="link_1" value="jaco_link_1" />
+	<property name="link_2" value="jaco_link_2" />
+	<property name="link_3" value="jaco_link_3" />
+	<property name="link_4" value="jaco_link_4" />
+	<property name="link_5" value="jaco_link_5" />
+	<property name="link_hand" value="jaco_link_hand" />
+	<property name="link_finger_1" value="jaco_link_finger_1" />
+	<property name="link_finger_2" value="jaco_link_finger_2" />
+	<property name="link_finger_3" value="jaco_link_finger_3" />
+	<property name="joint_base" value="jaco_joint_base" />
+	<property name="joint_base_axis_xyz" value="0 0 0" />
+	<property name="joint_base_origin_xyz" value="0 0 0" />
+	<property name="joint_base_origin_rpy" value="0 0 0" />
+	<property name="joint_1" value="jaco_joint_1" />
+	<property name="joint_1_axis_xyz" value="0 0 1" />
+	<property name="joint_1_origin_xyz" value="0 0 0.1535" />
+	<property name="joint_1_origin_rpy" value="${J_PI} 0 0" />
+	<property name="joint_2" value="jaco_joint_2" />
+	<property name="joint_2_axis_xyz" value="0 0 1" />
+	<property name="joint_2_origin_xyz" value="0 0 -0.1185" />
+	<property name="joint_2_origin_rpy" value="-${J_PI/2} -${J_PI/2} 0" />
+	<property name="joint_3" value="jaco_joint_3" />
+	<property name="joint_3_axis_xyz" value="0 0 1" />
+	<property name="joint_3_origin_xyz" value="0.41 0 0" />
+	<property name="joint_3_origin_rpy" value="${J_PI} 0 ${J_PI}" />
+	<property name="joint_4" value="jaco_joint_4" />
+	<property name="joint_4_axis_xyz" value="0 0 1" />
+	<property name="joint_4_origin_xyz" value="0.207 0 -0.01125" />
+	<property name="joint_4_origin_rpy" value="0 -${J_PI/2} 0" />
+	<property name="joint_5" value="jaco_joint_5" />
+	<property name="joint_5_axis_xyz" value="0 0 1" />
+	<property name="joint_5_origin_xyz" value="0.0343 0 -0.06588" />
+	<property name="joint_5_origin_rpy" value="0 ${J_PI/180*55} ${J_PI}" />
+	<property name="joint_6" value="jaco_joint_6" />
+	<property name="joint_6_axis_xyz" value="0 0 1" />
+	<property name="joint_6_origin_xyz" value="0.0343 0 -0.06588" />
+	<property name="joint_6_origin_rpy" value="0 ${J_PI/180*55} ${J_PI}" />
+	<property name="joint_finger_1" value="jaco_joint_finger_1" />
+	<property name="joint_finger_1_axis_xyz" value="0 0 1" />
+	<property name="joint_finger_1_origin_xyz" value="-0.03978 0 -0.10071" />
+	<property name="joint_finger_1_origin_rpy" value="-1.7983 1.117 3.1416" />
+	<property name="joint_finger_1_lower_limit" value="0" />
+	<property name="joint_finger_1_upper_limit" value="${J_PI/180*40}" />
+	<property name="joint_finger_2" value="jaco_joint_finger_2" />
+	<property name="joint_finger_2_axis_xyz" value="0 0 1" />
+	<property name="joint_finger_2_origin_xyz" value="0.03569 -0.0216 -0.10071" />
+	<property name="joint_finger_2_origin_rpy" value="-1.6222 1.117 -0.23615" />
+	<property name="joint_finger_2_lower_limit" value="0" />
+	<property name="joint_finger_2_upper_limit" value="${J_PI/180*40}" />
+	<property name="joint_finger_3" value="jaco_joint_finger_3" />
+	<property name="joint_finger_3_axis_xyz" value="0 0 1" />
+	<property name="joint_finger_3_origin_xyz" value="0.03569 0.0216 -0.10071" />
+	<property name="joint_finger_3_origin_rpy" value="-1.5161 1.1459 0.23978" />
+	<property name="joint_finger_3_lower_limit" value="0" />
+	<property name="joint_finger_3_upper_limit" value="${J_PI/180*40}" />
+	<xacro:macro name="jaco_link" params="link_name">
+		<link name="${link_name}">
+			<visual>
+				<geometry>
+					<mesh filename="package://jaco_model/meshes/${link_name}.dae" />
+				</geometry>
+				<material name="carbon_fiber">
+					<color rgba="0.792156862745098 0.819607843137255 0.933333333333333 1" />
+				</material>
+			</visual>
+			<collision>
+				<geometry>
+					<mesh filename="package://jaco_model/meshes/${link_name}.dae" />
+				</geometry>
+			</collision>
+		</link>
+	</xacro:macro>
+	<xacro:macro name="jaco_joint" params="joint_name type parent child joint_axis_xyz joint_origin_xyz joint_origin_rpy lower_limit upper_limit">
+		<joint name="${joint_name}" type="${type}">
+			<parent link="${parent}" />
+			<child link="${child}" />
+			<axis xyz="${joint_axis_xyz}" />
+			<origin xyz="${joint_origin_xyz}" rpy="${joint_origin_rpy}" />
+			<limit lower="${lower_limit}" upper="${upper_limit}" effort="30" velocity="5" />
+		</joint>
+	</xacro:macro>
+	<xacro:macro name="jaco_finger_joint" params="joint_name type parent child joint_axis_xyz joint_origin_xyz joint_origin_rpy lower_limit upper_limit">
+		<joint name="${joint_name}" type="${type}">
+			<parent link="${parent}" />
+			<child link="${child}" />
+			<axis xyz="${joint_axis_xyz}" />
+			<origin xyz="${joint_origin_xyz}" rpy="${joint_origin_rpy}" />
+			<limit lower="${lower_limit}" upper="${upper_limit}" effort="30" velocity="5" />
+		</joint>
+	</xacro:macro>
+	<xacro:macro name="jaco_arm" params="parent">
+		<xacro:jaco_link link_name="${link_base}" />
+		<xacro:jaco_joint joint_name="${joint_base}" type="fixed" parent="${parent}" child="${link_base}" joint_axis_xyz="${joint_base_axis_xyz}" joint_origin_xyz="${joint_base_origin_xyz}" joint_origin_rpy="${joint_base_origin_rpy}" lower_limit="-${J_LIM}" upper_limit="${J_LIM}" />
+		<xacro:jaco_link link_name="${link_1}" />
+		<xacro:jaco_joint joint_name="${joint_1}" type="revolute" parent="${link_base}" child="${link_1}" joint_axis_xyz="${joint_1_axis_xyz}" joint_origin_xyz="${joint_1_origin_xyz}" joint_origin_rpy="${joint_1_origin_rpy}" lower_limit="-${J_LIM}" upper_limit="${J_LIM}" />
+		<xacro:jaco_link link_name="${link_2}" />
+		<xacro:jaco_joint joint_name="${joint_2}" type="revolute" parent="${link_1}" child="${link_2}" joint_axis_xyz="${joint_2_axis_xyz}" joint_origin_xyz="${joint_2_origin_xyz}" joint_origin_rpy="${joint_2_origin_rpy}" lower_limit="0" upper_limit="${J_LIM}" />
+		<xacro:jaco_link link_name="${link_3}" />
+		<xacro:jaco_joint joint_name="${joint_3}" type="revolute" parent="${link_2}" child="${link_3}" joint_axis_xyz="${joint_3_axis_xyz}" joint_origin_xyz="${joint_3_origin_xyz}" joint_origin_rpy="${joint_3_origin_rpy}" lower_limit="0" upper_limit="${J_LIM}" />
+		<xacro:jaco_link link_name="${link_4}" />
+		<xacro:jaco_joint joint_name="${joint_4}" type="revolute" parent="${link_3}" child="${link_4}" joint_axis_xyz="${joint_4_axis_xyz}" joint_origin_xyz="${joint_4_origin_xyz}" joint_origin_rpy="${joint_4_origin_rpy}" lower_limit="-${J_LIM}" upper_limit="${J_LIM}" />
+		<xacro:jaco_link link_name="${link_5}" />
+		<xacro:jaco_joint joint_name="${joint_5}" type="revolute" parent="${link_4}" child="${link_5}" joint_axis_xyz="${joint_5_axis_xyz}" joint_origin_xyz="${joint_5_origin_xyz}" joint_origin_rpy="${joint_5_origin_rpy}" lower_limit="-${J_LIM}" upper_limit="${J_LIM}" />
+		<xacro:jaco_link link_name="${link_hand}" />
+		<xacro:jaco_joint joint_name="${joint_6}" type="revolute" parent="${link_5}" child="${link_hand}" joint_axis_xyz="${joint_6_axis_xyz}" joint_origin_xyz="${joint_6_origin_xyz}" joint_origin_rpy="${joint_6_origin_rpy}" lower_limit="-${J_LIM}" upper_limit="${J_LIM}" />
+		<xacro:jaco_link link_name="${link_finger_1}" />
+		<xacro:jaco_finger_joint joint_name="${joint_finger_1}" type="revolute" parent="${link_hand}" child="${link_finger_1}" joint_axis_xyz="${joint_finger_1_axis_xyz}" joint_origin_xyz="${joint_finger_1_origin_xyz}" joint_origin_rpy="${joint_finger_1_origin_rpy}" lower_limit="${joint_finger_1_lower_limit}" upper_limit="${joint_finger_1_upper_limit}" />
+		<xacro:jaco_link link_name="${link_finger_2}" />
+		<xacro:jaco_finger_joint joint_name="${joint_finger_2}" type="revolute" parent="${link_hand}" child="${link_finger_2}" joint_axis_xyz="${joint_finger_2_axis_xyz}" joint_origin_xyz="${joint_finger_2_origin_xyz}" joint_origin_rpy="${joint_finger_2_origin_rpy}" lower_limit="${joint_finger_2_lower_limit}" upper_limit="${joint_finger_2_upper_limit}" />
+		<xacro:jaco_link link_name="${link_finger_3}" />
+		<xacro:jaco_finger_joint joint_name="${joint_finger_3}" type="revolute" parent="${link_hand}" child="${link_finger_3}" joint_axis_xyz="${joint_finger_3_axis_xyz}" joint_origin_xyz="${joint_finger_3_origin_xyz}" joint_origin_rpy="${joint_finger_3_origin_rpy}" lower_limit="${joint_finger_3_lower_limit}" upper_limit="${joint_finger_3_upper_limit}" />
+	</xacro:macro>
 </root>

File: jaco_model/urdf/standalone_arm.xacro (robot description, xacro)
@@ -2,31 +2,30 @@
 <robot xmlns:xi="http://www.w3.org/2001/XInclude"
 	xmlns:gazebo="http://playerstage.sourceforge.net/gazebo/xmlschema/#gz"
-    xmlns:model="http://playerstage.sourceforge.net/gazebo/xmlschema/#model"
+	xmlns:model="http://playerstage.sourceforge.net/gazebo/xmlschema/#model"
 	xmlns:sensor="http://playerstage.sourceforge.net/gazebo/xmlschema/#sensor"
 	xmlns:body="http://playerstage.sourceforge.net/gazebo/xmlschema/#body"
-    xmlns:geom="http://playerstage.sourceforge.net/gazebo/xmlschema/#geom"
-    xmlns:joint="http://playerstage.sourceforge.net/gazebo/xmlschema/#joint"
+	xmlns:geom="http://playerstage.sourceforge.net/gazebo/xmlschema/#geom"
+	xmlns:joint="http://playerstage.sourceforge.net/gazebo/xmlschema/#joint"
 	xmlns:controller="http://playerstage.sourceforge.net/gazebo/xmlschema/#controller"
 	xmlns:interface="http://playerstage.sourceforge.net/gazebo/xmlschema/#interface"
 	xmlns:rendering="http://playerstage.sourceforge.net/gazebo/xmlschema/#rendering"
-    xmlns:renderable="http://playerstage.sourceforge.net/gazebo/xmlschema/#renderable"
-    xmlns:physics="http://playerstage.sourceforge.net/gazebo/xmlschema/#physics"
+	xmlns:renderable="http://playerstage.sourceforge.net/gazebo/xmlschema/#renderable"
+	xmlns:physics="http://playerstage.sourceforge.net/gazebo/xmlschema/#physics"
 	xmlns:xacro="http://ros.org/wiki/xacro" name="jaco">
-  <xacro:include filename="$(find jaco_model)/urdf/jaco_arm.xacro" />
-<link name="root">
-      <visual>
-	<origin xyz="0 0 0" rpy="0 0 0" />
-	<geometry>
-	  <box size = "0 0 0"/> <!--making it slightly bigger in x and z direction-->
-	</geometry>
-	<!--<material name="Black" /> -->
-      </visual>
-      <collision>
-	<origin xyz="0 0 0" rpy="0 0 0" />
-	<geometry>
-	  <box size = "0 0 0"/> <!--making it slightly bigger in x and z direction-->
-	</geometry>
-      </collision>
-    </link>
-<xacro:jaco_arm  parent="root"/>
+	<xacro:include filename="$(find jaco_model)/urdf/jaco_arm.xacro" />
+	<link name="root">
+		<visual>
+			<origin xyz="0 0 0" rpy="0 0 0" />
+			<geometry>
+				<box size = "0 0 0"/> <!-- making it slightly bigger in x and z direction -->
+			</geometry>
+		</visual>
+		<collision>
+			<origin xyz="0 0 0" rpy="0 0 0" />
+			<geometry>
+				<box size = "0 0 0"/> <!-- making it slightly bigger in x and z direction -->
+			</geometry>
+		</collision>
+	</link>
+	<xacro:jaco_arm parent="root" />
 </robot>
