Commit message: Updated xacro files to use jaco_description instead of jaco_model, generated urdf for standalone_arm

File: jaco_description/urdf/jaco_arm.xacro (robot description, xacro)
@@ -75,5 +75,5 @@
 			<visual>
 				<geometry>
-					<mesh filename="package://jaco_model/meshes/${link_name}.dae" />
+					<mesh filename="package://jaco_description/meshes/${link_name}.dae" />
 				</geometry>
 				<material name="carbon_fiber">
@@ -83,5 +83,5 @@
 			<collision>
 				<geometry>
-					<mesh filename="package://jaco_model/meshes/${link_name}.dae" />
+					<mesh filename="package://jaco_description/meshes/${link_name}.dae" />
 				</geometry>
 			</collision>

File: jaco_description/urdf/standalone_arm.xacro (robot description, xacro)
@@ -13,5 +13,5 @@
 	xmlns:physics="http://playerstage.sourceforge.net/gazebo/xmlschema/#physics"
 	xmlns:xacro="http://ros.org/wiki/xacro" name="jaco">
-	<xacro:include filename="$(find jaco_model)/urdf/jaco_arm.xacro" />
+	<xacro:include filename="$(find jaco_description)/urdf/jaco_arm.xacro" />
 	<link name="root">
 		<visual>

Commit message: Improved meshes and URDF

File: jaco_description/urdf/jaco_arm.xacro (robot description, xacro)
@@ -25,4 +25,7 @@
 	<property name="link_finger_2" value="jaco_link_finger_2" />
 	<property name="link_finger_3" value="jaco_link_finger_3" />
+	<property name="link_finger_tip_1" value="jaco_link_finger_tip_1" />
+	<property name="link_finger_tip_2" value="jaco_link_finger_tip_2" />
+	<property name="link_finger_tip_3" value="jaco_link_finger_tip_3" />
 	<property name="joint_base" value="jaco_joint_base" />
 	<property name="joint_base_axis_xyz" value="0 0 0" />
@@ -55,5 +58,5 @@
 	<property name="joint_finger_1" value="jaco_joint_finger_1" />
 	<property name="joint_finger_1_axis_xyz" value="0 0 1" />
-	<property name="joint_finger_1_origin_xyz" value="-0.03978 0 -0.10071" />
+	<property name="joint_finger_1_origin_xyz" value="-0.032578 0.0033 -0.12131" />
 	<property name="joint_finger_1_origin_rpy" value="-1.7983 1.117 3.1416" />
 	<property name="joint_finger_1_lower_limit" value="0" />
@@ -61,5 +64,5 @@
 	<property name="joint_finger_3" value="jaco_joint_finger_3" />
 	<property name="joint_finger_3_axis_xyz" value="0 0 1" />
-	<property name="joint_finger_3_origin_xyz" value="0.03569 -0.0216 -0.10071" />
+	<property name="joint_finger_3_origin_xyz" value="0.027788 -0.0206 -0.12131" />
 	<property name="joint_finger_3_origin_rpy" value="-1.6222 1.117 -0.23615" />
 	<property name="joint_finger_3_lower_limit" value="0" />
@@ -67,8 +70,26 @@
 	<property name="joint_finger_2" value="jaco_joint_finger_2" />
 	<property name="joint_finger_2_axis_xyz" value="0 0 1" />
-	<property name="joint_finger_2_origin_xyz" value="0.03569 0.0216 -0.10071" />
+	<property name="joint_finger_2_origin_xyz" value="0.027788 0.0206 -0.12131" />
 	<property name="joint_finger_2_origin_rpy" value="-1.5161 1.1459 0.23978" />
 	<property name="joint_finger_2_lower_limit" value="0" />
 	<property name="joint_finger_2_upper_limit" value="${J_PI/180*40}" />
+	<property name="joint_finger_tip_1" value="jaco_joint_finger_tip_1" />
+	<property name="joint_finger_tip_1_axis_xyz" value="0 0 1" />
+	<property name="joint_finger_tip_1_origin_xyz" value="0.044094 -0.0029 0" />
+	<property name="joint_finger_tip_1_origin_rpy" value="0 0 0" />
+	<property name="joint_finger_tip_1_lower_limit" value="0" />
+	<property name="joint_finger_tip_1_upper_limit" value="${J_PI/180*40}" />
+	<property name="joint_finger_tip_2" value="jaco_joint_finger_tip_2" />
+	<property name="joint_finger_tip_2_axis_xyz" value="0 0 1" />
+	<property name="joint_finger_tip_2_origin_xyz" value="0.044094 -0.0029 0" />
+	<property name="joint_finger_tip_2_origin_rpy" value="0 0 0" />
+	<property name="joint_finger_tip_2_lower_limit" value="0" />
+	<property name="joint_finger_tip_2_upper_limit" value="${J_PI/180*40}" />
+	<property name="joint_finger_tip_3" value="jaco_joint_finger_tip_3" />
+	<property name="joint_finger_tip_3_axis_xyz" value="0 0 1" />
+	<property name="joint_finger_tip_3_origin_xyz" value="0.044094 -0.0029 0" />
+	<property name="joint_finger_tip_3_origin_rpy" value="0 0 0" />
+	<property name="joint_finger_tip_3_lower_limit" value="0" />
+	<property name="joint_finger_tip_3_upper_limit" value="${J_PI/180*40}" />
 	<xacro:macro name="jaco_link" params="link_name">
 		<link name="${link_name}">
@@ -84,4 +105,21 @@
 				<geometry>
 					<mesh filename="package://jaco_description/meshes/${link_name}.dae" />
+				</geometry>
+			</collision>
+		</link>
+	</xacro:macro>
+	<xacro:macro name="ring_cover" params="suffix size">
+		<link name="${size}_ring_cover_${suffix}">
+			<visual>
+				<geometry>
+					<mesh filename="package://jaco_description/meshes/${size}_ring_cover.dae" />
+				</geometry>
+				<material name="carbon_fiber">
+					<color rgba="0.792156862745098 0.819607843137255 0.933333333333333 1" />
+				</material>
+			</visual>
+			<collision>
+				<geometry>
+					<mesh filename="package://jaco_description/meshes/${size}_ring_cover.dae" />
 				</geometry>
 			</collision>
@@ -121,4 +159,16 @@
 		<xacro:jaco_link link_name="${link_hand}" />
 		<xacro:jaco_joint joint_name="${joint_6}" type="revolute" parent="${link_5}" child="${link_hand}" joint_axis_xyz="${joint_6_axis_xyz}" joint_origin_xyz="${joint_6_origin_xyz}" joint_origin_rpy="${joint_6_origin_rpy}" lower_limit="-${J_LIM}" upper_limit="${J_LIM}" />
+		<xacro:ring_cover suffix="1" size="large"/>
+		<xacro:jaco_joint joint_name="large_ring_cover_1_joint" type="fixed" parent="${link_base}" child="large_ring_cover_1" joint_axis_xyz="${joint_1_axis_xyz}" joint_origin_xyz="${joint_1_origin_xyz}" joint_origin_rpy="${joint_1_origin_rpy}" lower_limit="-${J_LIM}" upper_limit="${J_LIM}" />
+		<xacro:ring_cover suffix="2" size="large"/>
+		<xacro:jaco_joint joint_name="large_ring_cover_2_joint" type="fixed" parent="${link_1}" child="large_ring_cover_2" joint_axis_xyz="${joint_2_axis_xyz}" joint_origin_xyz="${joint_2_origin_xyz}" joint_origin_rpy="${joint_2_origin_rpy}" lower_limit="0" upper_limit="${J_LIM}" />
+		<xacro:ring_cover suffix="3" size="large"/>
+		<xacro:jaco_joint joint_name="large_ring_cover_3_joint" type="fixed" parent="${link_2}" child="large_ring_cover_3" joint_axis_xyz="${joint_3_axis_xyz}" joint_origin_xyz="${joint_3_origin_xyz}" joint_origin_rpy="${joint_3_origin_rpy}" lower_limit="0" upper_limit="${J_LIM}" />
+		<xacro:ring_cover suffix="1" size="small"/>
+		<xacro:jaco_joint joint_name="large_ring_cover_4_joint" type="fixed" parent="${link_3}" child="small_ring_cover_1" joint_axis_xyz="${joint_4_axis_xyz}" joint_origin_xyz="${joint_4_origin_xyz}" joint_origin_rpy="${joint_4_origin_rpy}" lower_limit="-${J_LIM}" upper_limit="${J_LIM}" />
+		<xacro:ring_cover suffix="2" size="small"/>
+		<xacro:jaco_joint joint_name="large_ring_cover_5_joint" type="fixed" parent="${link_4}" child="small_ring_cover_2" joint_axis_xyz="${joint_5_axis_xyz}" joint_origin_xyz="${joint_5_origin_xyz}" joint_origin_rpy="${joint_5_origin_rpy}" lower_limit="-${J_LIM}" upper_limit="${J_LIM}" />
+		<xacro:ring_cover suffix="3" size="small"/>
+		<xacro:jaco_joint joint_name="large_ring_cover_6_joint" type="fixed" parent="${link_5}" child="small_ring_cover_3" joint_axis_xyz="${joint_6_axis_xyz}" joint_origin_xyz="${joint_6_origin_xyz}" joint_origin_rpy="${joint_6_origin_rpy}" lower_limit="-${J_LIM}" upper_limit="${J_LIM}" />
 		<xacro:jaco_link link_name="${link_finger_1}" />
 		<xacro:jaco_finger_joint joint_name="${joint_finger_1}" type="revolute" parent="${link_hand}" child="${link_finger_1}" joint_axis_xyz="${joint_finger_1_axis_xyz}" joint_origin_xyz="${joint_finger_1_origin_xyz}" joint_origin_rpy="${joint_finger_1_origin_rpy}" lower_limit="${joint_finger_1_lower_limit}" upper_limit="${joint_finger_1_upper_limit}" />
@@ -127,4 +177,10 @@
 		<xacro:jaco_link link_name="${link_finger_3}" />
 		<xacro:jaco_finger_joint joint_name="${joint_finger_3}" type="revolute" parent="${link_hand}" child="${link_finger_3}" joint_axis_xyz="${joint_finger_3_axis_xyz}" joint_origin_xyz="${joint_finger_3_origin_xyz}" joint_origin_rpy="${joint_finger_3_origin_rpy}" lower_limit="${joint_finger_3_lower_limit}" upper_limit="${joint_finger_3_upper_limit}" />
+		<xacro:jaco_link link_name="${link_finger_tip_1}" />
+		<xacro:jaco_finger_joint joint_name="${joint_finger_tip_1}" type="revolute" parent="${link_finger_1}" child="${link_finger_tip_1}" joint_axis_xyz="${joint_finger_tip_1_axis_xyz}" joint_origin_xyz="${joint_finger_tip_1_origin_xyz}" joint_origin_rpy="${joint_finger_tip_1_origin_rpy}" lower_limit="${joint_finger_tip_1_lower_limit}" upper_limit="${joint_finger_tip_1_upper_limit}" />
+		<xacro:jaco_link link_name="${link_finger_tip_2}" />
+		<xacro:jaco_finger_joint joint_name="${joint_finger_tip_2}" type="revolute" parent="${link_finger_2}" child="${link_finger_tip_2}" joint_axis_xyz="${joint_finger_tip_2_axis_xyz}" joint_origin_xyz="${joint_finger_tip_2_origin_xyz}" joint_origin_rpy="${joint_finger_tip_2_origin_rpy}" lower_limit="${joint_finger_tip_2_lower_limit}" upper_limit="${joint_finger_tip_2_upper_limit}" />
+		<xacro:jaco_link link_name="${link_finger_tip_3}" />
+		<xacro:jaco_finger_joint joint_name="${joint_finger_tip_3}" type="revolute" parent="${link_finger_3}" child="${link_finger_tip_3}" joint_axis_xyz="${joint_finger_tip_3_axis_xyz}" joint_origin_xyz="${joint_finger_tip_3_origin_xyz}" joint_origin_rpy="${joint_finger_tip_3_origin_rpy}" lower_limit="${joint_finger_tip_3_lower_limit}" upper_limit="${joint_finger_tip_3_upper_limit}" />
 	</xacro:macro>
 </root>

Commit message: Using low poly version of all meshes

File: jaco_description/urdf/jaco_arm.xacro (robot description, xacro)
@@ -109,9 +109,9 @@
 		</link>
 	</xacro:macro>
-	<xacro:macro name="ring_cover" params="suffix size">
-		<link name="${size}_ring_cover_${suffix}">
+	<xacro:macro name="jaco_ring_cover" params="suffix size">
+		<link name="jaco_${size}_ring_cover_${suffix}">
 			<visual>
 				<geometry>
-					<mesh filename="package://jaco_description/meshes/${size}_ring_cover.dae" />
+					<mesh filename="package://jaco_description/meshes/jaco_${size}_ring_cover.dae" />
 				</geometry>
 				<material name="carbon_fiber">
@@ -121,5 +121,5 @@
 			<collision>
 				<geometry>
-					<mesh filename="package://jaco_description/meshes/${size}_ring_cover.dae" />
+					<mesh filename="package://jaco_description/meshes/jaco_${size}_ring_cover.dae" />
 				</geometry>
 			</collision>
@@ -159,16 +159,16 @@
 		<xacro:jaco_link link_name="${link_hand}" />
 		<xacro:jaco_joint joint_name="${joint_6}" type="revolute" parent="${link_5}" child="${link_hand}" joint_axis_xyz="${joint_6_axis_xyz}" joint_origin_xyz="${joint_6_origin_xyz}" joint_origin_rpy="${joint_6_origin_rpy}" lower_limit="-${J_LIM}" upper_limit="${J_LIM}" />
-		<xacro:ring_cover suffix="1" size="large"/>
-		<xacro:jaco_joint joint_name="large_ring_cover_1_joint" type="fixed" parent="${link_base}" child="large_ring_cover_1" joint_axis_xyz="${joint_1_axis_xyz}" joint_origin_xyz="${joint_1_origin_xyz}" joint_origin_rpy="${joint_1_origin_rpy}" lower_limit="-${J_LIM}" upper_limit="${J_LIM}" />
-		<xacro:ring_cover suffix="2" size="large"/>
-		<xacro:jaco_joint joint_name="large_ring_cover_2_joint" type="fixed" parent="${link_1}" child="large_ring_cover_2" joint_axis_xyz="${joint_2_axis_xyz}" joint_origin_xyz="${joint_2_origin_xyz}" joint_origin_rpy="${joint_2_origin_rpy}" lower_limit="0" upper_limit="${J_LIM}" />
-		<xacro:ring_cover suffix="3" size="large"/>
-		<xacro:jaco_joint joint_name="large_ring_cover_3_joint" type="fixed" parent="${link_2}" child="large_ring_cover_3" joint_axis_xyz="${joint_3_axis_xyz}" joint_origin_xyz="${joint_3_origin_xyz}" joint_origin_rpy="${joint_3_origin_rpy}" lower_limit="0" upper_limit="${J_LIM}" />
-		<xacro:ring_cover suffix="1" size="small"/>
-		<xacro:jaco_joint joint_name="large_ring_cover_4_joint" type="fixed" parent="${link_3}" child="small_ring_cover_1" joint_axis_xyz="${joint_4_axis_xyz}" joint_origin_xyz="${joint_4_origin_xyz}" joint_origin_rpy="${joint_4_origin_rpy}" lower_limit="-${J_LIM}" upper_limit="${J_LIM}" />
-		<xacro:ring_cover suffix="2" size="small"/>
-		<xacro:jaco_joint joint_name="large_ring_cover_5_joint" type="fixed" parent="${link_4}" child="small_ring_cover_2" joint_axis_xyz="${joint_5_axis_xyz}" joint_origin_xyz="${joint_5_origin_xyz}" joint_origin_rpy="${joint_5_origin_rpy}" lower_limit="-${J_LIM}" upper_limit="${J_LIM}" />
-		<xacro:ring_cover suffix="3" size="small"/>
-		<xacro:jaco_joint joint_name="large_ring_cover_6_joint" type="fixed" parent="${link_5}" child="small_ring_cover_3" joint_axis_xyz="${joint_6_axis_xyz}" joint_origin_xyz="${joint_6_origin_xyz}" joint_origin_rpy="${joint_6_origin_rpy}" lower_limit="-${J_LIM}" upper_limit="${J_LIM}" />
+		<xacro:jaco_ring_cover suffix="1" size="large"/>
+		<xacro:jaco_joint joint_name="jaco_large_ring_cover_1_joint" type="fixed" parent="${link_base}" child="jaco_large_ring_cover_1" joint_axis_xyz="${joint_1_axis_xyz}" joint_origin_xyz="${joint_1_origin_xyz}" joint_origin_rpy="${joint_1_origin_rpy}" lower_limit="-${J_LIM}" upper_limit="${J_LIM}" />
+		<xacro:jaco_ring_cover suffix="2" size="large"/>
+		<xacro:jaco_joint joint_name="jaco_large_ring_cover_2_joint" type="fixed" parent="${link_1}" child="jaco_large_ring_cover_2" joint_axis_xyz="${joint_2_axis_xyz}" joint_origin_xyz="${joint_2_origin_xyz}" joint_origin_rpy="${joint_2_origin_rpy}" lower_limit="0" upper_limit="${J_LIM}" />
+		<xacro:jaco_ring_cover suffix="3" size="large"/>
+		<xacro:jaco_joint joint_name="jaco_large_ring_cover_3_joint" type="fixed" parent="${link_2}" child="jaco_large_ring_cover_3" joint_axis_xyz="${joint_3_axis_xyz}" joint_origin_xyz="${joint_3_origin_xyz}" joint_origin_rpy="${joint_3_origin_rpy}" lower_limit="0" upper_limit="${J_LIM}" />
+		<xacro:jaco_ring_cover suffix="1" size="small"/>
+		<xacro:jaco_joint joint_name="jaco_large_ring_cover_4_joint" type="fixed" parent="${link_3}" child="jaco_small_ring_cover_1" joint_axis_xyz="${joint_4_axis_xyz}" joint_origin_xyz="${joint_4_origin_xyz}" joint_origin_rpy="${joint_4_origin_rpy}" lower_limit="-${J_LIM}" upper_limit="${J_LIM}" />
+		<xacro:jaco_ring_cover suffix="2" size="small"/>
+		<xacro:jaco_joint joint_name="jaco_large_ring_cover_5_joint" type="fixed" parent="${link_4}" child="jaco_small_ring_cover_2" joint_axis_xyz="${joint_5_axis_xyz}" joint_origin_xyz="${joint_5_origin_xyz}" joint_origin_rpy="${joint_5_origin_rpy}" lower_limit="-${J_LIM}" upper_limit="${J_LIM}" />
+		<xacro:jaco_ring_cover suffix="3" size="small"/>
+		<xacro:jaco_joint joint_name="jaco_large_ring_cover_6_joint" type="fixed" parent="${link_5}" child="jaco_small_ring_cover_3" joint_axis_xyz="${joint_6_axis_xyz}" joint_origin_xyz="${joint_6_origin_xyz}" joint_origin_rpy="${joint_6_origin_rpy}" lower_limit="-${J_LIM}" upper_limit="${J_LIM}" />
 		<xacro:jaco_link link_name="${link_finger_1}" />
 		<xacro:jaco_finger_joint joint_name="${joint_finger_1}" type="revolute" parent="${link_hand}" child="${link_finger_1}" joint_axis_xyz="${joint_finger_1_axis_xyz}" joint_origin_xyz="${joint_finger_1_origin_xyz}" joint_origin_rpy="${joint_finger_1_origin_rpy}" lower_limit="${joint_finger_1_lower_limit}" upper_limit="${joint_finger_1_upper_limit}" />
