Commit message: Removed soft links

File: jaco_description/urdf/jaco_arm.xacro (robot description, xacro)
@@ -16,16 +16,11 @@
 	<property name="J_LIM" value="${2*J_PI}" />
 	<property name="link_base" value="jaco_link_base" />
+	<property name="link" value="jaco_link" />
 	<property name="link_1" value="jaco_link_1" />
 	<property name="link_2" value="jaco_link_2" />
 	<property name="link_3" value="jaco_link_3" />
-	<property name="link_4" value="jaco_link_4" />
-	<property name="link_5" value="jaco_link_5" />
 	<property name="link_hand" value="jaco_link_hand" />
-	<property name="link_finger_1" value="jaco_link_finger_1" />
-	<property name="link_finger_2" value="jaco_link_finger_2" />
-	<property name="link_finger_3" value="jaco_link_finger_3" />
-	<property name="link_finger_tip_1" value="jaco_link_finger_tip_1" />
-	<property name="link_finger_tip_2" value="jaco_link_finger_tip_2" />
-	<property name="link_finger_tip_3" value="jaco_link_finger_tip_3" />
+	<property name="link_finger" value="jaco_link_finger" />
+	<property name="link_finger_tip" value="jaco_link_finger_tip" />
 	<property name="joint_base" value="jaco_joint_base" />
 	<property name="joint_base_axis_xyz" value="0 0 0" />
@@ -109,4 +104,38 @@
 		</link>
 	</xacro:macro>
+	<xacro:macro name="jaco_link_suffix" params="link_name suffix">
+		<link name="${link_name}_${suffix}">
+			<visual>
+				<geometry>
+					<mesh filename="package://jaco_description/meshes/${link_name}.dae" />
+				</geometry>
+				<material name="carbon_fiber">
+					<color rgba="0.792156862745098 0.819607843137255 0.933333333333333 1" />
+				</material>
+			</visual>
+			<collision>
+				<geometry>
+					<mesh filename="package://jaco_description/meshes/${link_name}.dae" />
+				</geometry>
+			</collision>
+		</link>
+	</xacro:macro>
+	<xacro:macro name="jaco_link_4_5" params="link_name suffix">
+		<link name="${link_name}_${suffix}">
+			<visual>
+				<geometry>
+					<mesh filename="package://jaco_description/meshes/${link_name}_4_5.dae" />
+				</geometry>
+				<material name="carbon_fiber">
+					<color rgba="0.792156862745098 0.819607843137255 0.933333333333333 1" />
+				</material>
+			</visual>
+			<collision>
+				<geometry>
+					<mesh filename="package://jaco_description/meshes/${link_name}_4_5.dae" />
+				</geometry>
+			</collision>
+		</link>
+	</xacro:macro>
 	<xacro:macro name="jaco_ring_cover" params="suffix size">
 		<link name="jaco_${size}_ring_cover_${suffix}">
@@ -153,10 +182,10 @@
 		<xacro:jaco_link link_name="${link_3}" />
 		<xacro:jaco_joint joint_name="${joint_3}" type="revolute" parent="${link_2}" child="${link_3}" joint_axis_xyz="${joint_3_axis_xyz}" joint_origin_xyz="${joint_3_origin_xyz}" joint_origin_rpy="${joint_3_origin_rpy}" lower_limit="0" upper_limit="${J_LIM}" />
-		<xacro:jaco_link link_name="${link_4}" />
-		<xacro:jaco_joint joint_name="${joint_4}" type="revolute" parent="${link_3}" child="${link_4}" joint_axis_xyz="${joint_4_axis_xyz}" joint_origin_xyz="${joint_4_origin_xyz}" joint_origin_rpy="${joint_4_origin_rpy}" lower_limit="-${J_LIM}" upper_limit="${J_LIM}" />
-		<xacro:jaco_link link_name="${link_5}" />
-		<xacro:jaco_joint joint_name="${joint_5}" type="revolute" parent="${link_4}" child="${link_5}" joint_axis_xyz="${joint_5_axis_xyz}" joint_origin_xyz="${joint_5_origin_xyz}" joint_origin_rpy="${joint_5_origin_rpy}" lower_limit="-${J_LIM}" upper_limit="${J_LIM}" />
+		<xacro:jaco_link_4_5 link_name="${link}" suffix="4"/>
+		<xacro:jaco_joint joint_name="${joint_4}" type="revolute" parent="${link_3}" child="${link}_4" joint_axis_xyz="${joint_4_axis_xyz}" joint_origin_xyz="${joint_4_origin_xyz}" joint_origin_rpy="${joint_4_origin_rpy}" lower_limit="-${J_LIM}" upper_limit="${J_LIM}" />
+		<xacro:jaco_link_4_5 link_name="${link}" suffix="5"/>
+		<xacro:jaco_joint joint_name="${joint_5}" type="revolute" parent="${link}_4" child="${link}_5" joint_axis_xyz="${joint_5_axis_xyz}" joint_origin_xyz="${joint_5_origin_xyz}" joint_origin_rpy="${joint_5_origin_rpy}" lower_limit="-${J_LIM}" upper_limit="${J_LIM}" />
 		<xacro:jaco_link link_name="${link_hand}" />
-		<xacro:jaco_joint joint_name="${joint_6}" type="revolute" parent="${link_5}" child="${link_hand}" joint_axis_xyz="${joint_6_axis_xyz}" joint_origin_xyz="${joint_6_origin_xyz}" joint_origin_rpy="${joint_6_origin_rpy}" lower_limit="-${J_LIM}" upper_limit="${J_LIM}" />
+		<xacro:jaco_joint joint_name="${joint_6}" type="revolute" parent="${link}_5" child="${link_hand}" joint_axis_xyz="${joint_6_axis_xyz}" joint_origin_xyz="${joint_6_origin_xyz}" joint_origin_rpy="${joint_6_origin_rpy}" lower_limit="-${J_LIM}" upper_limit="${J_LIM}" />
 		<xacro:jaco_ring_cover suffix="1" size="large"/>
 		<xacro:jaco_joint joint_name="jaco_large_ring_cover_1_joint" type="fixed" parent="${link_base}" child="jaco_large_ring_cover_1" joint_axis_xyz="${joint_1_axis_xyz}" joint_origin_xyz="${joint_1_origin_xyz}" joint_origin_rpy="${joint_1_origin_rpy}" lower_limit="-${J_LIM}" upper_limit="${J_LIM}" />
@@ -168,19 +197,19 @@
 		<xacro:jaco_joint joint_name="jaco_large_ring_cover_4_joint" type="fixed" parent="${link_3}" child="jaco_small_ring_cover_1" joint_axis_xyz="${joint_4_axis_xyz}" joint_origin_xyz="${joint_4_origin_xyz}" joint_origin_rpy="${joint_4_origin_rpy}" lower_limit="-${J_LIM}" upper_limit="${J_LIM}" />
 		<xacro:jaco_ring_cover suffix="2" size="small"/>
-		<xacro:jaco_joint joint_name="jaco_large_ring_cover_5_joint" type="fixed" parent="${link_4}" child="jaco_small_ring_cover_2" joint_axis_xyz="${joint_5_axis_xyz}" joint_origin_xyz="${joint_5_origin_xyz}" joint_origin_rpy="${joint_5_origin_rpy}" lower_limit="-${J_LIM}" upper_limit="${J_LIM}" />
+		<xacro:jaco_joint joint_name="jaco_large_ring_cover_5_joint" type="fixed" parent="${link}_4" child="jaco_small_ring_cover_2" joint_axis_xyz="${joint_5_axis_xyz}" joint_origin_xyz="${joint_5_origin_xyz}" joint_origin_rpy="${joint_5_origin_rpy}" lower_limit="-${J_LIM}" upper_limit="${J_LIM}" />
 		<xacro:jaco_ring_cover suffix="3" size="small"/>
-		<xacro:jaco_joint joint_name="jaco_large_ring_cover_6_joint" type="fixed" parent="${link_5}" child="jaco_small_ring_cover_3" joint_axis_xyz="${joint_6_axis_xyz}" joint_origin_xyz="${joint_6_origin_xyz}" joint_origin_rpy="${joint_6_origin_rpy}" lower_limit="-${J_LIM}" upper_limit="${J_LIM}" />
-		<xacro:jaco_link link_name="${link_finger_1}" />
-		<xacro:jaco_finger_joint joint_name="${joint_finger_1}" type="revolute" parent="${link_hand}" child="${link_finger_1}" joint_axis_xyz="${joint_finger_1_axis_xyz}" joint_origin_xyz="${joint_finger_1_origin_xyz}" joint_origin_rpy="${joint_finger_1_origin_rpy}" lower_limit="${joint_finger_1_lower_limit}" upper_limit="${joint_finger_1_upper_limit}" />
-		<xacro:jaco_link link_name="${link_finger_2}" />
-		<xacro:jaco_finger_joint joint_name="${joint_finger_2}" type="revolute" parent="${link_hand}" child="${link_finger_2}" joint_axis_xyz="${joint_finger_2_axis_xyz}" joint_origin_xyz="${joint_finger_2_origin_xyz}" joint_origin_rpy="${joint_finger_2_origin_rpy}" lower_limit="${joint_finger_2_lower_limit}" upper_limit="${joint_finger_2_upper_limit}" />
-		<xacro:jaco_link link_name="${link_finger_3}" />
-		<xacro:jaco_finger_joint joint_name="${joint_finger_3}" type="revolute" parent="${link_hand}" child="${link_finger_3}" joint_axis_xyz="${joint_finger_3_axis_xyz}" joint_origin_xyz="${joint_finger_3_origin_xyz}" joint_origin_rpy="${joint_finger_3_origin_rpy}" lower_limit="${joint_finger_3_lower_limit}" upper_limit="${joint_finger_3_upper_limit}" />
-		<xacro:jaco_link link_name="${link_finger_tip_1}" />
-		<xacro:jaco_finger_joint joint_name="${joint_finger_tip_1}" type="revolute" parent="${link_finger_1}" child="${link_finger_tip_1}" joint_axis_xyz="${joint_finger_tip_1_axis_xyz}" joint_origin_xyz="${joint_finger_tip_1_origin_xyz}" joint_origin_rpy="${joint_finger_tip_1_origin_rpy}" lower_limit="${joint_finger_tip_1_lower_limit}" upper_limit="${joint_finger_tip_1_upper_limit}" />
-		<xacro:jaco_link link_name="${link_finger_tip_2}" />
-		<xacro:jaco_finger_joint joint_name="${joint_finger_tip_2}" type="revolute" parent="${link_finger_2}" child="${link_finger_tip_2}" joint_axis_xyz="${joint_finger_tip_2_axis_xyz}" joint_origin_xyz="${joint_finger_tip_2_origin_xyz}" joint_origin_rpy="${joint_finger_tip_2_origin_rpy}" lower_limit="${joint_finger_tip_2_lower_limit}" upper_limit="${joint_finger_tip_2_upper_limit}" />
-		<xacro:jaco_link link_name="${link_finger_tip_3}" />
-		<xacro:jaco_finger_joint joint_name="${joint_finger_tip_3}" type="revolute" parent="${link_finger_3}" child="${link_finger_tip_3}" joint_axis_xyz="${joint_finger_tip_3_axis_xyz}" joint_origin_xyz="${joint_finger_tip_3_origin_xyz}" joint_origin_rpy="${joint_finger_tip_3_origin_rpy}" lower_limit="${joint_finger_tip_3_lower_limit}" upper_limit="${joint_finger_tip_3_upper_limit}" />
+		<xacro:jaco_joint joint_name="jaco_large_ring_cover_6_joint" type="fixed" parent="${link}_4" child="jaco_small_ring_cover_3" joint_axis_xyz="${joint_6_axis_xyz}" joint_origin_xyz="${joint_6_origin_xyz}" joint_origin_rpy="${joint_6_origin_rpy}" lower_limit="-${J_LIM}" upper_limit="${J_LIM}" />
+		<xacro:jaco_link_suffix link_name="${link_finger}" suffix="1"/>
+		<xacro:jaco_finger_joint joint_name="${joint_finger_1}" type="revolute" parent="${link_hand}" child="${link_finger}_1" joint_axis_xyz="${joint_finger_1_axis_xyz}" joint_origin_xyz="${joint_finger_1_origin_xyz}" joint_origin_rpy="${joint_finger_1_origin_rpy}" lower_limit="${joint_finger_1_lower_limit}" upper_limit="${joint_finger_1_upper_limit}" />
+		<xacro:jaco_link_suffix link_name="${link_finger}" suffix="2"/>
+		<xacro:jaco_finger_joint joint_name="${joint_finger_2}" type="revolute" parent="${link_hand}" child="${link_finger}_2" joint_axis_xyz="${joint_finger_2_axis_xyz}" joint_origin_xyz="${joint_finger_2_origin_xyz}" joint_origin_rpy="${joint_finger_2_origin_rpy}" lower_limit="${joint_finger_2_lower_limit}" upper_limit="${joint_finger_2_upper_limit}" />
+		<xacro:jaco_link_suffix link_name="${link_finger}" suffix="3"/>
+		<xacro:jaco_finger_joint joint_name="${joint_finger_3}" type="revolute" parent="${link_hand}" child="${link_finger}_3" joint_axis_xyz="${joint_finger_3_axis_xyz}" joint_origin_xyz="${joint_finger_3_origin_xyz}" joint_origin_rpy="${joint_finger_3_origin_rpy}" lower_limit="${joint_finger_3_lower_limit}" upper_limit="${joint_finger_3_upper_limit}" />
+		<xacro:jaco_link_suffix link_name="${link_finger_tip}" suffix="1"/>
+		<xacro:jaco_finger_joint joint_name="${joint_finger_tip_1}" type="revolute" parent="${link_finger}_1" child="${link_finger_tip}_1" joint_axis_xyz="${joint_finger_tip_1_axis_xyz}" joint_origin_xyz="${joint_finger_tip_1_origin_xyz}" joint_origin_rpy="${joint_finger_tip_1_origin_rpy}" lower_limit="${joint_finger_tip_1_lower_limit}" upper_limit="${joint_finger_tip_1_upper_limit}" />
+		<xacro:jaco_link_suffix link_name="${link_finger_tip}" suffix="2"/>
+		<xacro:jaco_finger_joint joint_name="${joint_finger_tip_2}" type="revolute" parent="${link_finger}_2" child="${link_finger_tip}_2" joint_axis_xyz="${joint_finger_tip_2_axis_xyz}" joint_origin_xyz="${joint_finger_tip_2_origin_xyz}" joint_origin_rpy="${joint_finger_tip_2_origin_rpy}" lower_limit="${joint_finger_tip_2_lower_limit}" upper_limit="${joint_finger_tip_2_upper_limit}" />
+		<xacro:jaco_link_suffix link_name="${link_finger_tip}" suffix="3"/>
+		<xacro:jaco_finger_joint joint_name="${joint_finger_tip_3}" type="revolute" parent="${link_finger}_3" child="${link_finger_tip}_3" joint_axis_xyz="${joint_finger_tip_3_axis_xyz}" joint_origin_xyz="${joint_finger_tip_3_origin_xyz}" joint_origin_rpy="${joint_finger_tip_3_origin_rpy}" lower_limit="${joint_finger_tip_3_lower_limit}" upper_limit="${joint_finger_tip_3_upper_limit}" />
 	</xacro:macro>
 </root>

Commit message: fixed URDF to load minified files

File: jaco_description/urdf/jaco_arm.xacro (robot description, xacro)
@@ -91,13 +91,13 @@
 			<visual>
 				<geometry>
-					<mesh filename="package://jaco_description/meshes/${link_name}.dae" />
-				</geometry>
-				<material name="carbon_fiber">
-					<color rgba="0.792156862745098 0.819607843137255 0.933333333333333 1" />
-				</material>
-			</visual>
-			<collision>
-				<geometry>
-					<mesh filename="package://jaco_description/meshes/${link_name}.dae" />
+					<mesh filename="package://jaco_description/meshes/${link_name}.min.dae" />
+				</geometry>
+				<material name="carbon_fiber">
+					<color rgba="0.792156862745098 0.819607843137255 0.933333333333333 1" />
+				</material>
+			</visual>
+			<collision>
+				<geometry>
+					<mesh filename="package://jaco_description/meshes/${link_name}.min.dae" />
 				</geometry>
 			</collision>
@@ -108,13 +108,13 @@
 			<visual>
 				<geometry>
-					<mesh filename="package://jaco_description/meshes/${link_name}.dae" />
-				</geometry>
-				<material name="carbon_fiber">
-					<color rgba="0.792156862745098 0.819607843137255 0.933333333333333 1" />
-				</material>
-			</visual>
-			<collision>
-				<geometry>
-					<mesh filename="package://jaco_description/meshes/${link_name}.dae" />
+					<mesh filename="package://jaco_description/meshes/${link_name}.min.dae" />
+				</geometry>
+				<material name="carbon_fiber">
+					<color rgba="0.792156862745098 0.819607843137255 0.933333333333333 1" />
+				</material>
+			</visual>
+			<collision>
+				<geometry>
+					<mesh filename="package://jaco_description/meshes/${link_name}.min.dae" />
 				</geometry>
 			</collision>
@@ -125,13 +125,13 @@
 			<visual>
 				<geometry>
-					<mesh filename="package://jaco_description/meshes/${link_name}_4_5.dae" />
-				</geometry>
-				<material name="carbon_fiber">
-					<color rgba="0.792156862745098 0.819607843137255 0.933333333333333 1" />
-				</material>
-			</visual>
-			<collision>
-				<geometry>
-					<mesh filename="package://jaco_description/meshes/${link_name}_4_5.dae" />
+					<mesh filename="package://jaco_description/meshes/${link_name}_4_5.min.dae" />
+				</geometry>
+				<material name="carbon_fiber">
+					<color rgba="0.792156862745098 0.819607843137255 0.933333333333333 1" />
+				</material>
+			</visual>
+			<collision>
+				<geometry>
+					<mesh filename="package://jaco_description/meshes/${link_name}_4_5.min.dae" />
 				</geometry>
 			</collision>
@@ -142,13 +142,13 @@
 			<visual>
 				<geometry>
-					<mesh filename="package://jaco_description/meshes/jaco_${size}_ring_cover.dae" />
-				</geometry>
-				<material name="carbon_fiber">
-					<color rgba="0.792156862745098 0.819607843137255 0.933333333333333 1" />
-				</material>
-			</visual>
-			<collision>
-				<geometry>
-					<mesh filename="package://jaco_description/meshes/jaco_${size}_ring_cover.dae" />
+					<mesh filename="package://jaco_description/meshes/jaco_${size}_ring_cover.min.dae" />
+				</geometry>
+				<material name="carbon_fiber">
+					<color rgba="0.792156862745098 0.819607843137255 0.933333333333333 1" />
+				</material>
+			</visual>
+			<collision>
+				<geometry>
+					<mesh filename="package://jaco_description/meshes/jaco_${size}_ring_cover.min.dae" />
 				</geometry>
 			</collision>
