Commit message: updated pre-compiled URDF

File: jaco_description/urdf/standalone_arm.urdf (robot description, URDF)
Before this commit: robot jaco, 11 links, 10 joints
Links:
- added link jaco_large_ring_cover_1; collision mesh filename=package://jaco_description/meshes/jaco_large_ring_cover.dae; visual mesh filename=package://jaco_description/meshes/jaco_large_ring_cover.dae
- added link jaco_large_ring_cover_2; collision mesh filename=package://jaco_description/meshes/jaco_large_ring_cover.dae; visual mesh filename=package://jaco_description/meshes/jaco_large_ring_cover.dae
- added link jaco_large_ring_cover_3; collision mesh filename=package://jaco_description/meshes/jaco_large_ring_cover.dae; visual mesh filename=package://jaco_description/meshes/jaco_large_ring_cover.dae
- added link jaco_link_finger_tip_1; collision mesh filename=package://jaco_description/meshes/jaco_link_finger_tip.dae; visual mesh filename=package://jaco_description/meshes/jaco_link_finger_tip.dae
- added link jaco_link_finger_tip_2; collision mesh filename=package://jaco_description/meshes/jaco_link_finger_tip.dae; visual mesh filename=package://jaco_description/meshes/jaco_link_finger_tip.dae
- added link jaco_link_finger_tip_3; collision mesh filename=package://jaco_description/meshes/jaco_link_finger_tip.dae; visual mesh filename=package://jaco_description/meshes/jaco_link_finger_tip.dae
- added link jaco_small_ring_cover_1; collision mesh filename=package://jaco_description/meshes/jaco_small_ring_cover.dae; visual mesh filename=package://jaco_description/meshes/jaco_small_ring_cover.dae
- added link jaco_small_ring_cover_2; collision mesh filename=package://jaco_description/meshes/jaco_small_ring_cover.dae; visual mesh filename=package://jaco_description/meshes/jaco_small_ring_cover.dae
- added link jaco_small_ring_cover_3; collision mesh filename=package://jaco_description/meshes/jaco_small_ring_cover.dae; visual mesh filename=package://jaco_description/meshes/jaco_small_ring_cover.dae
- link jaco_link_4: geometry collision mesh filename=package://jaco_description/meshes/jaco_link_4_5.dae; visual mesh filename=package://jaco_description/meshes/jaco_link_4_5.dae
- link jaco_link_5: geometry collision mesh filename=package://jaco_description/meshes/jaco_link_4_5.dae; visual mesh filename=package://jaco_description/meshes/jaco_link_4_5.dae
- link jaco_link_finger_1: geometry collision mesh filename=package://jaco_description/meshes/jaco_link_finger.dae; visual mesh filename=package://jaco_description/meshes/jaco_link_finger.dae
- link jaco_link_finger_2: geometry collision mesh filename=package://jaco_description/meshes/jaco_link_finger.dae; visual mesh filename=package://jaco_description/meshes/jaco_link_finger.dae
- link jaco_link_finger_3: geometry collision mesh filename=package://jaco_description/meshes/jaco_link_finger.dae; visual mesh filename=package://jaco_description/meshes/jaco_link_finger.dae
Joints:
- added joint jaco_joint_finger_tip_1: type revolute, parent jaco_link_finger_1, child jaco_link_finger_tip_1, origin xyz=0.044094 -0.0029 0 rpy=0 0 0, axis 0 0 1, limit lower=0 upper=0.698131700798 effort=30 velocity=5
- added joint jaco_joint_finger_tip_2: type revolute, parent jaco_link_finger_2, child jaco_link_finger_tip_2, origin xyz=0.044094 -0.0029 0 rpy=0 0 0, axis 0 0 1, limit lower=0 upper=0.698131700798 effort=30 velocity=5
- added joint jaco_joint_finger_tip_3: type revolute, parent jaco_link_finger_3, child jaco_link_finger_tip_3, origin xyz=0.044094 -0.0029 0 rpy=0 0 0, axis 0 0 1, limit lower=0 upper=0.698131700798 effort=30 velocity=5
- added joint jaco_large_ring_cover_1_joint: type fixed, parent jaco_link_base, child jaco_large_ring_cover_1, origin xyz=0 0 0.1535 rpy=3.14159265359 0 0, axis 0 0 1, limit lower=-6.28318530718 upper=6.28318530718 effort=30 velocity=5
- added joint jaco_large_ring_cover_2_joint: type fixed, parent jaco_link_1, child jaco_large_ring_cover_2, origin xyz=0 0 -0.1185 rpy=-1.57079632679 -1.57079632679 0, axis 0 0 1, limit lower=0 upper=6.28318530718 effort=30 velocity=5
- added joint jaco_large_ring_cover_3_joint: type fixed, parent jaco_link_2, child jaco_large_ring_cover_3, origin xyz=0.41 0 0 rpy=3.14159265359 0 3.14159265359, axis 0 0 1, limit lower=0 upper=6.28318530718 effort=30 velocity=5
- added joint jaco_large_ring_cover_4_joint: type fixed, parent jaco_link_3, child jaco_small_ring_cover_1, origin xyz=0.207 0 -0.01125 rpy=0 -1.57079632679 0, axis 0 0 1, limit lower=-6.28318530718 upper=6.28318530718 effort=30 velocity=5
- added joint jaco_large_ring_cover_5_joint: type fixed, parent jaco_link_4, child jaco_small_ring_cover_2, origin xyz=0.0343 0 -0.06588 rpy=0 0.959931088597 3.14159265359, axis 0 0 1, limit lower=-6.28318530718 upper=6.28318530718 effort=30 velocity=5
- added joint jaco_large_ring_cover_6_joint: type fixed, parent jaco_link_4, child jaco_small_ring_cover_3, origin xyz=0.0343 0 -0.06588 rpy=0 0.959931088597 3.14159265359, axis 0 0 1, limit lower=-6.28318530718 upper=6.28318530718 effort=30 velocity=5
- joint jaco_joint_finger_1: origin xyz=-0.03978 0 -0.10071 rpy=-1.7983 1.117 3.1416 -> xyz=-0.032578 0.0033 -0.12131 rpy=-1.7983 1.117 3.1416
- joint jaco_joint_finger_2: origin xyz=0.03569 0.0216 -0.10071 rpy=-1.5161 1.1459 0.23978 -> xyz=0.027788 0.0206 -0.12131 rpy=-1.5161 1.1459 0.23978
- joint jaco_joint_finger_3: origin xyz=0.03569 -0.0216 -0.10071 rpy=-1.6222 1.117 -0.23615 -> xyz=0.027788 -0.0206 -0.12131 rpy=-1.6222 1.117 -0.23615

Commit message: recompiled URDF

File: jaco_description/urdf/standalone_arm.urdf (robot description, URDF)
Before this commit: robot jaco, 20 links, 19 joints
Links:
- link jaco_large_ring_cover_1: geometry collision mesh filename=package://jaco_description/meshes/jaco_large_ring_cover.min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; visual mesh filename=package://jaco_description/meshes/jaco_large_ring_cover.min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
- link jaco_large_ring_cover_2: geometry collision mesh filename=package://jaco_description/meshes/jaco_large_ring_cover.min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; visual mesh filename=package://jaco_description/meshes/jaco_large_ring_cover.min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
- link jaco_large_ring_cover_3: geometry collision mesh filename=package://jaco_description/meshes/jaco_large_ring_cover.min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; visual mesh filename=package://jaco_description/meshes/jaco_large_ring_cover.min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
- link jaco_link_1: geometry collision mesh filename=package://jaco_description/meshes/jaco_link_1.min.dae; visual mesh filename=package://jaco_description/meshes/jaco_link_1.min.dae
- link jaco_link_2: geometry collision mesh filename=package://jaco_description/meshes/jaco_link_2.min.dae; visual mesh filename=package://jaco_description/meshes/jaco_link_2.min.dae
- link jaco_link_3: geometry collision mesh filename=package://jaco_description/meshes/jaco_link_3.min.dae; visual mesh filename=package://jaco_description/meshes/jaco_link_3.min.dae
- link jaco_link_4: geometry collision mesh filename=package://jaco_description/meshes/jaco_link_4_5.min.dae; visual mesh filename=package://jaco_description/meshes/jaco_link_4_5.min.dae
- link jaco_link_5: geometry collision mesh filename=package://jaco_description/meshes/jaco_link_4_5.min.dae; visual mesh filename=package://jaco_description/meshes/jaco_link_4_5.min.dae
- link jaco_link_base: geometry collision mesh filename=package://jaco_description/meshes/jaco_link_base.min.dae; visual mesh filename=package://jaco_description/meshes/jaco_link_base.min.dae
- link jaco_link_finger_1: geometry collision mesh filename=package://jaco_description/meshes/jaco_link_finger.min.dae; visual mesh filename=package://jaco_description/meshes/jaco_link_finger.min.dae
- link jaco_link_finger_2: geometry collision mesh filename=package://jaco_description/meshes/jaco_link_finger.min.dae; visual mesh filename=package://jaco_description/meshes/jaco_link_finger.min.dae
- link jaco_link_finger_3: geometry collision mesh filename=package://jaco_description/meshes/jaco_link_finger.min.dae; visual mesh filename=package://jaco_description/meshes/jaco_link_finger.min.dae
- link jaco_link_finger_tip_1: geometry collision mesh filename=package://jaco_description/meshes/jaco_link_finger_tip.min.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; visual mesh filename=package://jaco_description/meshes/jaco_link_finger_tip.min.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
- link jaco_link_finger_tip_2: geometry collision mesh filename=package://jaco_description/meshes/jaco_link_finger_tip.min.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; visual mesh filename=package://jaco_description/meshes/jaco_link_finger_tip.min.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
- link jaco_link_finger_tip_3: geometry collision mesh filename=package://jaco_description/meshes/jaco_link_finger_tip.min.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; visual mesh filename=package://jaco_description/meshes/jaco_link_finger_tip.min.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
- link jaco_link_hand: geometry collision mesh filename=package://jaco_description/meshes/jaco_link_hand.min.dae; visual mesh filename=package://jaco_description/meshes/jaco_link_hand.min.dae
- link jaco_small_ring_cover_1: geometry collision mesh filename=package://jaco_description/meshes/jaco_small_ring_cover.min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; visual mesh filename=package://jaco_description/meshes/jaco_small_ring_cover.min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
- link jaco_small_ring_cover_2: geometry collision mesh filename=package://jaco_description/meshes/jaco_small_ring_cover.min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; visual mesh filename=package://jaco_description/meshes/jaco_small_ring_cover.min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
- link jaco_small_ring_cover_3: geometry collision mesh filename=package://jaco_description/meshes/jaco_small_ring_cover.min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; visual mesh filename=package://jaco_description/meshes/jaco_small_ring_cover.min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
