Commit message: minified XML

File: jaco_description/urdf/jaco_arm.urdf.xacro (robot description, xacro)
@@ -92,5 +92,5 @@
 			<visual>
 				<geometry>
-					<mesh scale="${M_SCALE} ${M_SCALE} ${M_SCALE}" filename="package://jaco_description/meshes/${link_name}.dae" />
+					<mesh scale="${M_SCALE} ${M_SCALE} ${M_SCALE}" filename="package://jaco_description/meshes/${link_name}.min.dae" />
 				</geometry>
 				<material name="carbon_fiber">
@@ -109,5 +109,5 @@
 			<visual>
 				<geometry>
-					<mesh scale="${M_SCALE} ${M_SCALE} ${M_SCALE}" filename="package://jaco_description/meshes/${link_name}.dae" />
+					<mesh scale="${M_SCALE} ${M_SCALE} ${M_SCALE}" filename="package://jaco_description/meshes/${link_name}.min.dae" />
 				</geometry>
 				<material name="carbon_fiber">
@@ -126,5 +126,5 @@
 			<visual>
 				<geometry>
-					<mesh scale="${M_SCALE} ${M_SCALE} ${M_SCALE}" filename="package://jaco_description/meshes/${link_name}_4_5.dae" />
+					<mesh scale="${M_SCALE} ${M_SCALE} ${M_SCALE}" filename="package://jaco_description/meshes/${link_name}_4_5.min.dae" />
 				</geometry>
 				<material name="carbon_fiber">
@@ -143,5 +143,5 @@
 			<visual>
 				<geometry>
-					<mesh scale="${M_SCALE} ${M_SCALE} ${M_SCALE}" filename="package://jaco_description/meshes/jaco_${size}_ring_cover.dae" />
+					<mesh scale="${M_SCALE} ${M_SCALE} ${M_SCALE}" filename="package://jaco_description/meshes/jaco_${size}_ring_cover.min.dae" />
 				</geometry>
 				<material name="carbon_fiber">

Commit message: Added Gazebo support.
Added necessary elements for Gazebo simulation:
- Mass (currently made up)
- Inertia (currently made up)
- Joint controllers for the Gazebo robot using ROS Control
- Transmissions on necessary joints
- Gripper tag to support grasping (may need tuning)

File: jaco_description/urdf/jaco_arm.urdf.xacro (robot description, xacro)
@@ -88,4 +88,9 @@
 	<xacro:macro name="jaco_link" params="link_name">
 		<link name="${link_name}">
+            <inertial>
+                <mass value="1"/>
+                <inertia ixx="0.1" ixy="0" ixz="0" iyy="0.1" iyz="0" izz="0.1"/>
+                <origin/>
+            </inertial>
 			<visual>
 				<geometry>
@@ -105,4 +110,9 @@
 	<xacro:macro name="jaco_link_suffix" params="link_name suffix">
 		<link name="${link_name}_${suffix}">
+            <inertial>
+                <mass value="0.25"/>
+                <inertia ixx="0.01" ixy="0" ixz="0" iyy="0.01" iyz="0" izz="0.01"/>
+                <origin/>
+            </inertial>
 			<visual>
 				<geometry>
@@ -122,4 +132,9 @@
 	<xacro:macro name="jaco_link_4_5" params="link_name suffix">
 		<link name="${link_name}_${suffix}">
+            <inertial>
+                <mass value="0.5"/>
+                <inertia ixx="0.01" ixy="0" ixz="0" iyy="0.01" iyz="0" izz="0.01"/>
+                <origin/>
+            </inertial>
 			<visual>
 				<geometry>
@@ -139,4 +154,9 @@
 	<xacro:macro name="jaco_ring_cover" params="suffix size">
 		<link name="jaco_${size}_ring_cover_${suffix}">
+            <inertial>
+                <mass value="0"/>
+                <inertia ixx="0" ixy="0" ixz="0" iyy="0" iyz="0" izz="0"/>
+                <origin/>
+            </inertial>
 			<visual>
 				<geometry>
@@ -172,19 +192,42 @@
 		</joint>
 	</xacro:macro>
+	<xacro:macro name="jaco_transmission" params="joint_name">
+        <transmission name="${joint_name}_transmission">
+            <type>transmission_interface/SimpleTransmission</type>
+            <joint name="${joint_name}">
+              <hardwareInterface>PositionJointInterface</hardwareInterface>
+            </joint>
+            <actuator name="${joint_name}_motor">
+              <mechanicalReduction>1</mechanicalReduction>
+            </actuator>
+        </transmission>
+	</xacro:macro>
 	<xacro:macro name="jaco_arm" params="parent xyz rpy">
+        <gazebo>
+            <plugin filename="libgazebo_ros_control.so" name="gazebo_ros_controller_manager">
+                <!-- <robotNamespace>/</robotNamespace> -->
+                <robotParam>robot_description</robotParam>
+            </plugin>
+        </gazebo>
 		<xacro:jaco_link link_name="${link_base}" />
 		<xacro:jaco_joint joint_name="${joint_base}" type="fixed" parent="${parent}" child="${link_base}" joint_axis_xyz="${joint_base_axis_xyz}" joint_origin_xyz="${xyz}" joint_origin_rpy="${rpy}" lower_limit="-${J_LIM}" upper_limit="${J_LIM}" />
 		<xacro:jaco_link link_name="${link_1}" />
 		<xacro:jaco_joint joint_name="${joint_1}" type="revolute" parent="${link_base}" child="${link_1}" joint_axis_xyz="${joint_1_axis_xyz}" joint_origin_xyz="${joint_1_origin_xyz}" joint_origin_rpy="${joint_1_origin_rpy}" lower_limit="-${J_LIM}" upper_limit="${J_LIM}" />
+        <xacro:jaco_transmission joint_name="${joint_1}" />
 		<xacro:jaco_link link_name="${link_2}" />
 		<xacro:jaco_joint joint_name="${joint_2}" type="revolute" parent="${link_1}" child="${link_2}" joint_axis_xyz="${joint_2_axis_xyz}" joint_origin_xyz="${joint_2_origin_xyz}" joint_origin_rpy="${joint_2_origin_rpy}" lower_limit="0" upper_limit="${J_LIM}" />
+        <xacro:jaco_transmission joint_name="${joint_2}" />
 		<xacro:jaco_link link_name="${link_3}" />
 		<xacro:jaco_joint joint_name="${joint_3}" type="revolute" parent="${link_2}" child="${link_3}" joint_axis_xyz="${joint_3_axis_xyz}" joint_origin_xyz="${joint_3_origin_xyz}" joint_origin_rpy="${joint_3_origin_rpy}" lower_limit="0" upper_limit="${J_LIM}" />
+        <xacro:jaco_transmission joint_name="${joint_3}" />
 		<xacro:jaco_link_4_5 link_name="${link}" suffix="4"/>
 		<xacro:jaco_joint joint_name="${joint_4}" type="revolute" parent="${link_3}" child="${link}_4" joint_axis_xyz="${joint_4_axis_xyz}" joint_origin_xyz="${joint_4_origin_xyz}" joint_origin_rpy="${joint_4_origin_rpy}" lower_limit="-${J_LIM}" upper_limit="${J_LIM}" />
+        <xacro:jaco_transmission joint_name="${joint_4}" />
 		<xacro:jaco_link_4_5 link_name="${link}" suffix="5"/>
 		<xacro:jaco_joint joint_name="${joint_5}" type="revolute" parent="${link}_4" child="${link}_5" joint_axis_xyz="${joint_5_axis_xyz}" joint_origin_xyz="${joint_5_origin_xyz}" joint_origin_rpy="${joint_5_origin_rpy}" lower_limit="-${J_LIM}" upper_limit="${J_LIM}" />
+        <xacro:jaco_transmission joint_name="${joint_5}" />
 		<xacro:jaco_link link_name="${link_hand}" />
 		<xacro:jaco_joint joint_name="${joint_6}" type="revolute" parent="${link}_5" child="${link_hand}" joint_axis_xyz="${joint_6_axis_xyz}" joint_origin_xyz="${joint_6_origin_xyz}" joint_origin_rpy="${joint_6_origin_rpy}" lower_limit="-${J_LIM}" upper_limit="${J_LIM}" />
+        <xacro:jaco_transmission joint_name="${joint_6}" />
 		<xacro:jaco_ring_cover suffix="1" size="large"/>
 		<xacro:jaco_joint joint_name="jaco_large_ring_cover_1_joint" type="fixed" parent="${link_base}" child="jaco_large_ring_cover_1" joint_axis_xyz="${joint_1_axis_xyz}" joint_origin_xyz="${joint_1_origin_xyz}" joint_origin_rpy="${joint_1_origin_rpy}" lower_limit="-${J_LIM}" upper_limit="${J_LIM}" />
@@ -201,14 +244,38 @@
 		<xacro:jaco_link_suffix link_name="${link_finger}" suffix="1"/>
 		<xacro:jaco_finger_joint joint_name="${joint_finger_1}" type="revolute" parent="${link_hand}" child="${link_finger}_1" joint_axis_xyz="${joint_finger_1_axis_xyz}" joint_origin_xyz="${joint_finger_1_origin_xyz}" joint_origin_rpy="${joint_finger_1_origin_rpy}" lower_limit="${joint_finger_1_lower_limit}" upper_limit="${joint_finger_1_upper_limit}" />
+        <xacro:jaco_transmission joint_name="${joint_finger_1}" />
 		<xacro:jaco_link_suffix link_name="${link_finger}" suffix="2"/>
 		<xacro:jaco_finger_joint joint_name="${joint_finger_2}" type="revolute" parent="${link_hand}" child="${link_finger}_2" joint_axis_xyz="${joint_finger_2_axis_xyz}" joint_origin_xyz="${joint_finger_2_origin_xyz}" joint_origin_rpy="${joint_finger_2_origin_rpy}" lower_limit="${joint_finger_2_lower_limit}" upper_limit="${joint_finger_2_upper_limit}" />
+        <xacro:jaco_transmission joint_name="${joint_finger_2}" />
 		<xacro:jaco_link_suffix link_name="${link_finger}" suffix="3"/>
 		<xacro:jaco_finger_joint joint_name="${joint_finger_3}" type="revolute" parent="${link_hand}" child="${link_finger}_3" joint_axis_xyz="${joint_finger_3_axis_xyz}" joint_origin_xyz="${joint_finger_3_origin_xyz}" joint_origin_rpy="${joint_finger_3_origin_rpy}" lower_limit="${joint_finger_3_lower_limit}" upper_limit="${joint_finger_3_upper_limit}" />
+        <xacro:jaco_transmission joint_name="${joint_finger_3}" />
 		<xacro:jaco_link_suffix link_name="${link_finger_tip}" suffix="1"/>
 		<xacro:jaco_finger_joint joint_name="${joint_finger_tip_1}" type="revolute" parent="${link_finger}_1" child="${link_finger_tip}_1" joint_axis_xyz="${joint_finger_tip_1_axis_xyz}" joint_origin_xyz="${joint_finger_tip_1_origin_xyz}" joint_origin_rpy="${joint_finger_tip_1_origin_rpy}" lower_limit="${joint_finger_tip_1_lower_limit}" upper_limit="${joint_finger_tip_1_upper_limit}" />
+        <xacro:jaco_transmission joint_name="${joint_finger_tip_1}" />
 		<xacro:jaco_link_suffix link_name="${link_finger_tip}" suffix="2"/>
 		<xacro:jaco_finger_joint joint_name="${joint_finger_tip_2}" type="revolute" parent="${link_finger}_2" child="${link_finger_tip}_2" joint_axis_xyz="${joint_finger_tip_2_axis_xyz}" joint_origin_xyz="${joint_finger_tip_2_origin_xyz}" joint_origin_rpy="${joint_finger_tip_2_origin_rpy}" lower_limit="${joint_finger_tip_2_lower_limit}" upper_limit="${joint_finger_tip_2_upper_limit}" />
+        <xacro:jaco_transmission joint_name="${joint_finger_tip_2}" />
 		<xacro:jaco_link_suffix link_name="${link_finger_tip}" suffix="3"/>
 		<xacro:jaco_finger_joint joint_name="${joint_finger_tip_3}" type="revolute" parent="${link_finger}_3" child="${link_finger_tip}_3" joint_axis_xyz="${joint_finger_tip_3_axis_xyz}" joint_origin_xyz="${joint_finger_tip_3_origin_xyz}" joint_origin_rpy="${joint_finger_tip_3_origin_rpy}" lower_limit="${joint_finger_tip_3_lower_limit}" upper_limit="${joint_finger_tip_3_upper_limit}" />
+        <xacro:jaco_transmission joint_name="${joint_finger_tip_3}" />
+        <gazebo>
+          <gripper name="grasping">
+            <grasp_check>
+              <attach_steps>5</attach_steps>
+              <detach_steps>20</detach_steps>
+              <min_contact_count>1</min_contact_count>
+            </grasp_check>
+            <gripper_link>${link_finger}_1</gripper_link>
+            <gripper_link>${link_finger}_2</gripper_link>
+            <gripper_link>${link_finger}_3</gripper_link>
+            <gripper_link>${link_finger_tip}_1</gripper_link>
+            <gripper_link>${link_finger_tip}_2</gripper_link>
+            <gripper_link>${link_finger_tip}_3</gripper_link>
+            <palm_link>${link_hand}</palm_link>
+            <!-- <gripper_link>${link_hand}</gripper_link> -->
+            <!-- <palm_link>${link_finger_tip}_1</palm_link> -->
+          </gripper>
+        </gazebo>
 	</xacro:macro>
 </robot>
