Commit message: rebuild of URDF

File: jaco_description/robots/standalone_arm.urdf (robot description, URDF)
Before this commit: robot jaco, 20 links, 19 joints
Links:
- link jaco_large_ring_cover_1: geometry collision mesh filename=package://jaco_description/meshes/jaco_large_ring_cover.stl scale=0.0254 0.0254 0.0254; visual mesh filename=package://jaco_description/meshes/jaco_large_ring_cover.min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 scale=0.0254 0.0254 0.0254
- link jaco_large_ring_cover_2: geometry collision mesh filename=package://jaco_description/meshes/jaco_large_ring_cover.stl scale=0.0254 0.0254 0.0254; visual mesh filename=package://jaco_description/meshes/jaco_large_ring_cover.min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 scale=0.0254 0.0254 0.0254
- link jaco_large_ring_cover_3: geometry collision mesh filename=package://jaco_description/meshes/jaco_large_ring_cover.stl scale=0.0254 0.0254 0.0254; visual mesh filename=package://jaco_description/meshes/jaco_large_ring_cover.min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 scale=0.0254 0.0254 0.0254
- link jaco_link_1: geometry collision mesh filename=package://jaco_description/meshes/jaco_link_1.stl scale=0.0254 0.0254 0.0254; visual mesh filename=package://jaco_description/meshes/jaco_link_1.min.dae scale=0.0254 0.0254 0.0254
- link jaco_link_2: geometry collision mesh filename=package://jaco_description/meshes/jaco_link_2.stl scale=0.0254 0.0254 0.0254; visual mesh filename=package://jaco_description/meshes/jaco_link_2.min.dae scale=0.0254 0.0254 0.0254
- link jaco_link_3: geometry collision mesh filename=package://jaco_description/meshes/jaco_link_3.stl scale=0.0254 0.0254 0.0254; visual mesh filename=package://jaco_description/meshes/jaco_link_3.min.dae scale=0.0254 0.0254 0.0254
- link jaco_link_4: geometry collision mesh filename=package://jaco_description/meshes/jaco_link_4_5.stl scale=0.0254 0.0254 0.0254; visual mesh filename=package://jaco_description/meshes/jaco_link_4_5.min.dae scale=0.0254 0.0254 0.0254
- link jaco_link_5: geometry collision mesh filename=package://jaco_description/meshes/jaco_link_4_5.stl scale=0.0254 0.0254 0.0254; visual mesh filename=package://jaco_description/meshes/jaco_link_4_5.min.dae scale=0.0254 0.0254 0.0254
- link jaco_link_base: geometry collision mesh filename=package://jaco_description/meshes/jaco_link_base.stl scale=0.0254 0.0254 0.0254; visual mesh filename=package://jaco_description/meshes/jaco_link_base.min.dae scale=0.0254 0.0254 0.0254
- link jaco_link_finger_1: geometry collision mesh filename=package://jaco_description/meshes/jaco_link_finger.stl scale=0.0254 0.0254 0.0254; visual mesh filename=package://jaco_description/meshes/jaco_link_finger.min.dae scale=0.0254 0.0254 0.0254
- link jaco_link_finger_2: geometry collision mesh filename=package://jaco_description/meshes/jaco_link_finger.stl scale=0.0254 0.0254 0.0254; visual mesh filename=package://jaco_description/meshes/jaco_link_finger.min.dae scale=0.0254 0.0254 0.0254
- link jaco_link_finger_3: geometry collision mesh filename=package://jaco_description/meshes/jaco_link_finger.stl scale=0.0254 0.0254 0.0254; visual mesh filename=package://jaco_description/meshes/jaco_link_finger.min.dae scale=0.0254 0.0254 0.0254
- link jaco_link_finger_tip_1: geometry collision mesh filename=package://jaco_description/meshes/jaco_link_finger_tip.stl scale=0.0254 0.0254 0.0254; visual mesh filename=package://jaco_description/meshes/jaco_link_finger_tip.min.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 scale=0.0254 0.0254 0.0254
- link jaco_link_finger_tip_2: geometry collision mesh filename=package://jaco_description/meshes/jaco_link_finger_tip.stl scale=0.0254 0.0254 0.0254; visual mesh filename=package://jaco_description/meshes/jaco_link_finger_tip.min.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 scale=0.0254 0.0254 0.0254
- link jaco_link_finger_tip_3: geometry collision mesh filename=package://jaco_description/meshes/jaco_link_finger_tip.stl scale=0.0254 0.0254 0.0254; visual mesh filename=package://jaco_description/meshes/jaco_link_finger_tip.min.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 scale=0.0254 0.0254 0.0254
- link jaco_link_hand: geometry collision mesh filename=package://jaco_description/meshes/jaco_link_hand.stl scale=0.0254 0.0254 0.0254; visual mesh filename=package://jaco_description/meshes/jaco_link_hand.min.dae scale=0.0254 0.0254 0.0254
- link jaco_small_ring_cover_1: geometry collision mesh filename=package://jaco_description/meshes/jaco_small_ring_cover.stl scale=0.0254 0.0254 0.0254; visual mesh filename=package://jaco_description/meshes/jaco_small_ring_cover.min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 scale=0.0254 0.0254 0.0254
- link jaco_small_ring_cover_2: geometry collision mesh filename=package://jaco_description/meshes/jaco_small_ring_cover.stl scale=0.0254 0.0254 0.0254; visual mesh filename=package://jaco_description/meshes/jaco_small_ring_cover.min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 scale=0.0254 0.0254 0.0254
- link jaco_small_ring_cover_3: geometry collision mesh filename=package://jaco_description/meshes/jaco_small_ring_cover.stl scale=0.0254 0.0254 0.0254; visual mesh filename=package://jaco_description/meshes/jaco_small_ring_cover.min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 scale=0.0254 0.0254 0.0254
Joints:
- joint jaco_joint_3: origin xyz=0.41 0 0 rpy=3.14159265359 0 3.14159265359 -> xyz=0.41 0 0 rpy=0 0 3.14159265359
- joint jaco_large_ring_cover_3_joint: origin xyz=0.41 0 0 rpy=3.14159265359 0 3.14159265359 -> xyz=0.41 0 0 rpy=0 0 3.14159265359

Commit message: Updated urdf and regenerated urdf file

File: jaco_description/robots/standalone_arm.urdf (robot description, URDF)
Before this commit: robot jaco, 20 links, 19 joints
Joints:
- joint jaco_joint_3: origin xyz=0.41 0 0 rpy=0 0 3.14159265359 -> xyz=0.41 0 0 rpy=3.14159265359 0 3.14159265359
- joint jaco_large_ring_cover_3_joint: origin xyz=0.41 0 0 rpy=0 0 3.14159265359 -> xyz=0.41 0 0 rpy=3.14159265359 0 3.14159265359
- joint jaco_large_ring_cover_6_joint: parent jaco_link_4 -> jaco_link_5

File: jaco_description/urdf/jaco_arm.urdf.xacro (robot description, xacro)
@@ -39,5 +39,5 @@
 	<xacro:property name="joint_3_axis_xyz" value="0 0 1" />
 	<xacro:property name="joint_3_origin_xyz" value="0.41 0 0" />
-	<xacro:property name="joint_3_origin_rpy" value="0 0 ${M_PI}" />
+	<xacro:property name="joint_3_origin_rpy" value="${M_PI} 0 ${M_PI}" />
 	<xacro:property name="joint_4" value="jaco_joint_4" />
 	<xacro:property name="joint_4_axis_xyz" value="0 0 1" />
@@ -200,5 +200,5 @@
 		<xacro:jaco_joint joint_name="jaco_large_ring_cover_5_joint" type="fixed" parent="${link}_4" child="jaco_small_ring_cover_2" joint_axis_xyz="${joint_5_axis_xyz}" joint_origin_xyz="${joint_5_origin_xyz}" joint_origin_rpy="${joint_5_origin_rpy}" lower_limit="-${J_LIM}" upper_limit="${J_LIM}" />
 		<xacro:jaco_ring_cover suffix="3" size="small"/>
-		<xacro:jaco_joint joint_name="jaco_large_ring_cover_6_joint" type="fixed" parent="${link}_4" child="jaco_small_ring_cover_3" joint_axis_xyz="${joint_6_axis_xyz}" joint_origin_xyz="${joint_6_origin_xyz}" joint_origin_rpy="${joint_6_origin_rpy}" lower_limit="-${J_LIM}" upper_limit="${J_LIM}" />
+		<xacro:jaco_joint joint_name="jaco_large_ring_cover_6_joint" type="fixed" parent="${link}_5" child="jaco_small_ring_cover_3" joint_axis_xyz="${joint_6_axis_xyz}" joint_origin_xyz="${joint_6_origin_xyz}" joint_origin_rpy="${joint_6_origin_rpy}" lower_limit="-${J_LIM}" upper_limit="${J_LIM}" />
 		<xacro:jaco_link_suffix link_name="${link_finger}" suffix="1"/>
 		<xacro:jaco_finger_joint joint_name="${joint_finger_1}" type="revolute" parent="${link_hand}" child="${link_finger}_1" joint_axis_xyz="${joint_finger_1_axis_xyz}" joint_origin_xyz="${joint_finger_1_origin_xyz}" joint_origin_rpy="${joint_finger_1_origin_rpy}" lower_limit="${joint_finger_1_lower_limit}" upper_limit="${joint_finger_1_upper_limit}" />

Commit message: fixed start position of arm

File: jaco_description/robots/standalone_arm.urdf (robot description, URDF)
Before this commit: robot jaco, 20 links, 19 joints
Joints:
- joint jaco_joint_1: origin xyz=0 0 0.1535 rpy=3.14159265359 0 0 -> xyz=0 0 0.1535 rpy=3.14159265359 0 1.412
- joint jaco_joint_2: origin xyz=0 0 -0.1185 rpy=-1.57079632679 -1.57079632679 0 -> xyz=0 0 -0.1185 rpy=-1.57079632679 1.403 0
- joint jaco_joint_3: origin xyz=0.41 0 0 rpy=3.14159265359 0 3.14159265359 -> xyz=0.41 0 0 rpy=-3.14159265359 0 2.274
- joint jaco_joint_4: origin xyz=0.207 0 -0.01125 rpy=0 -1.57079632679 0 -> xyz=0.207 0 -0.01125 rpy=1.57079632679 0.752 -1.57079632679
- joint jaco_joint_5: origin xyz=0.0343 0 -0.06588 rpy=0 0.959931088597 3.14159265359 -> xyz=0.0343 0 -0.06588 rpy=0.959 -0.045 -1.539
- joint jaco_joint_6: origin xyz=0.0343 0 -0.06588 rpy=0 0.959931088597 3.14159265359 -> xyz=0.0343 0 -0.06588 rpy=0.953 0.139 -1.669
- joint jaco_large_ring_cover_1_joint: origin xyz=0 0 0.1535 rpy=3.14159265359 0 0 -> xyz=0 0 0.1535 rpy=3.14159265359 0 1.412
- joint jaco_large_ring_cover_2_joint: origin xyz=0 0 -0.1185 rpy=-1.57079632679 -1.57079632679 0 -> xyz=0 0 -0.1185 rpy=-1.57079632679 1.403 0
- joint jaco_large_ring_cover_3_joint: origin xyz=0.41 0 0 rpy=3.14159265359 0 3.14159265359 -> xyz=0.41 0 0 rpy=-3.14159265359 0 2.274
- joint jaco_large_ring_cover_4_joint: origin xyz=0.207 0 -0.01125 rpy=0 -1.57079632679 0 -> xyz=0.207 0 -0.01125 rpy=1.57079632679 0.752 -1.57079632679
- joint jaco_large_ring_cover_5_joint: origin xyz=0.0343 0 -0.06588 rpy=0 0.959931088597 3.14159265359 -> xyz=0.0343 0 -0.06588 rpy=0.959 -0.045 -1.539
- joint jaco_large_ring_cover_6_joint: origin xyz=0.0343 0 -0.06588 rpy=0 0.959931088597 3.14159265359 -> xyz=0.0343 0 -0.06588 rpy=0.953 0.139 -1.669

File: jaco_description/robots/standalone_arm.urdf.xacro (robot description, xacro)
@@ -28,4 +28,4 @@
 		</collision>
 	</link>
-	<xacro:jaco_arm parent="root" />
+	<xacro:jaco_arm parent="root" xyz="0 0 0" rpy="0 0 0" />
 </robot>

File: jaco_description/urdf/jaco_arm.urdf.xacro (robot description, xacro)
@@ -26,30 +26,28 @@
 	<xacro:property name="joint_base" value="jaco_joint_base" />
 	<xacro:property name="joint_base_axis_xyz" value="0 0 0" />
-	<xacro:property name="joint_base_origin_xyz" value="0 0 0" />
-	<xacro:property name="joint_base_origin_rpy" value="0 0 0" />
 	<xacro:property name="joint_1" value="jaco_joint_1" />
 	<xacro:property name="joint_1_axis_xyz" value="0 0 1" />
 	<xacro:property name="joint_1_origin_xyz" value="0 0 0.1535" />
-	<xacro:property name="joint_1_origin_rpy" value="${M_PI} 0 0" />
+	<xacro:property name="joint_1_origin_rpy" value="${M_PI} 0 1.412" />
 	<xacro:property name="joint_2" value="jaco_joint_2" />
 	<xacro:property name="joint_2_axis_xyz" value="0 0 1" />
 	<xacro:property name="joint_2_origin_xyz" value="0 0 -0.1185" />
-	<xacro:property name="joint_2_origin_rpy" value="-${M_PI/2} -${M_PI/2} 0" />
+	<xacro:property name="joint_2_origin_rpy" value="-${M_PI/2} 1.403 0" />
 	<xacro:property name="joint_3" value="jaco_joint_3" />
 	<xacro:property name="joint_3_axis_xyz" value="0 0 1" />
 	<xacro:property name="joint_3_origin_xyz" value="0.41 0 0" />
-	<xacro:property name="joint_3_origin_rpy" value="${M_PI} 0 ${M_PI}" />
+	<xacro:property name="joint_3_origin_rpy" value="-${M_PI} 0 2.274" />
 	<xacro:property name="joint_4" value="jaco_joint_4" />
 	<xacro:property name="joint_4_axis_xyz" value="0 0 1" />
 	<xacro:property name="joint_4_origin_xyz" value="0.207 0 -0.01125" />
-	<xacro:property name="joint_4_origin_rpy" value="0 -${M_PI/2} 0" />
+	<xacro:property name="joint_4_origin_rpy" value="${M_PI/2} 0.752 -${M_PI/2}" />
 	<xacro:property name="joint_5" value="jaco_joint_5" />
 	<xacro:property name="joint_5_axis_xyz" value="0 0 1" />
 	<xacro:property name="joint_5_origin_xyz" value="0.0343 0 -0.06588" />
-	<xacro:property name="joint_5_origin_rpy" value="0 ${M_PI/180*55} ${M_PI}" />
+	<xacro:property name="joint_5_origin_rpy" value="0.959 -0.045 -1.539" />
 	<xacro:property name="joint_6" value="jaco_joint_6" />
 	<xacro:property name="joint_6_axis_xyz" value="0 0 1" />
 	<xacro:property name="joint_6_origin_xyz" value="0.0343 0 -0.06588" />
-	<xacro:property name="joint_6_origin_rpy" value="0 ${M_PI/180*55} ${M_PI}" />
+	<xacro:property name="joint_6_origin_rpy" value="0.953 0.139 -1.669" />
 	<xacro:property name="joint_finger_1" value="jaco_joint_finger_1" />
 	<xacro:property name="joint_finger_1_axis_xyz" value="0 0 1" />
@@ -174,7 +172,7 @@
 		</joint>
 	</xacro:macro>
-	<xacro:macro name="jaco_arm" params="parent">
+	<xacro:macro name="jaco_arm" params="parent xyz rpy">
 		<xacro:jaco_link link_name="${link_base}" />
-		<xacro:jaco_joint joint_name="${joint_base}" type="fixed" parent="${parent}" child="${link_base}" joint_axis_xyz="${joint_base_axis_xyz}" joint_origin_xyz="${joint_base_origin_xyz}" joint_origin_rpy="${joint_base_origin_rpy}" lower_limit="-${J_LIM}" upper_limit="${J_LIM}" />
+		<xacro:jaco_joint joint_name="${joint_base}" type="fixed" parent="${parent}" child="${link_base}" joint_axis_xyz="${joint_base_axis_xyz}" joint_origin_xyz="${xyz}" joint_origin_rpy="${rpy}" lower_limit="-${J_LIM}" upper_limit="${J_LIM}" />
 		<xacro:jaco_link link_name="${link_1}" />
 		<xacro:jaco_joint joint_name="${joint_1}" type="revolute" parent="${link_base}" child="${link_1}" joint_axis_xyz="${joint_1_axis_xyz}" joint_origin_xyz="${joint_1_origin_xyz}" joint_origin_rpy="${joint_1_origin_rpy}" lower_limit="-${J_LIM}" upper_limit="${J_LIM}" />
