Commit message: start position fixed

File: jaco_description/robots/standalone_arm.urdf (robot description, URDF)
Before this commit: robot jaco, 20 links, 19 joints
Joints:
- joint jaco_joint_1: origin xyz=0 0 0.1535 rpy=3.14159265359 0 1.412 -> xyz=0 0 0.1535 rpy=3.14159265359 0 0
- joint jaco_joint_2: origin xyz=0 0 -0.1185 rpy=-1.57079632679 1.403 0 -> xyz=0 0 -0.1185 rpy=-1.57079632679 -1.57079632679 0
- joint jaco_joint_3: origin xyz=0.41 0 0 rpy=-3.14159265359 0 2.274 -> xyz=0.41 0 0 rpy=3.14159265359 0 3.14159265359
- joint jaco_joint_4: origin xyz=0.207 0 -0.01125 rpy=1.57079632679 0.752 -1.57079632679 -> xyz=0.207 0 -0.01125 rpy=0 -1.57079632679 0
- joint jaco_joint_5: origin xyz=0.0343 0 -0.06588 rpy=0.959 -0.045 -1.539 -> xyz=0.0343 0 -0.06588 rpy=0 0.959931088597 3.14159265359
- joint jaco_joint_6: origin xyz=0.0343 0 -0.06588 rpy=0.953 0.139 -1.669 -> xyz=0.0343 0 -0.06588 rpy=0 0.959931088597 3.14159265359
- joint jaco_large_ring_cover_1_joint: origin xyz=0 0 0.1535 rpy=3.14159265359 0 1.412 -> xyz=0 0 0.1535 rpy=3.14159265359 0 0
- joint jaco_large_ring_cover_2_joint: origin xyz=0 0 -0.1185 rpy=-1.57079632679 1.403 0 -> xyz=0 0 -0.1185 rpy=-1.57079632679 -1.57079632679 0
- joint jaco_large_ring_cover_3_joint: origin xyz=0.41 0 0 rpy=-3.14159265359 0 2.274 -> xyz=0.41 0 0 rpy=3.14159265359 0 3.14159265359
- joint jaco_large_ring_cover_4_joint: origin xyz=0.207 0 -0.01125 rpy=1.57079632679 0.752 -1.57079632679 -> xyz=0.207 0 -0.01125 rpy=0 -1.57079632679 0
- joint jaco_large_ring_cover_5_joint: origin xyz=0.0343 0 -0.06588 rpy=0.959 -0.045 -1.539 -> xyz=0.0343 0 -0.06588 rpy=0 0.959931088597 3.14159265359
- joint jaco_large_ring_cover_6_joint: origin xyz=0.0343 0 -0.06588 rpy=0.953 0.139 -1.669 -> xyz=0.0343 0 -0.06588 rpy=0 0.959931088597 3.14159265359

File: jaco_description/urdf/jaco_arm.urdf.xacro (robot description, xacro)
@@ -27,63 +27,63 @@
 	<xacro:property name="joint_base_axis_xyz" value="0 0 0" />
 	<xacro:property name="joint_1" value="jaco_joint_1" />
-	<xacro:property name="joint_1_axis_xyz" value="0 0 1" />
-	<xacro:property name="joint_1_origin_xyz" value="0 0 0.1535" />
-	<xacro:property name="joint_1_origin_rpy" value="${M_PI} 0 1.412" />
-	<xacro:property name="joint_2" value="jaco_joint_2" />
-	<xacro:property name="joint_2_axis_xyz" value="0 0 1" />
-	<xacro:property name="joint_2_origin_xyz" value="0 0 -0.1185" />
-	<xacro:property name="joint_2_origin_rpy" value="-${M_PI/2} 1.403 0" />
-	<xacro:property name="joint_3" value="jaco_joint_3" />
-	<xacro:property name="joint_3_axis_xyz" value="0 0 1" />
-	<xacro:property name="joint_3_origin_xyz" value="0.41 0 0" />
-	<xacro:property name="joint_3_origin_rpy" value="-${M_PI} 0 2.274" />
-	<xacro:property name="joint_4" value="jaco_joint_4" />
-	<xacro:property name="joint_4_axis_xyz" value="0 0 1" />
-	<xacro:property name="joint_4_origin_xyz" value="0.207 0 -0.01125" />
-	<xacro:property name="joint_4_origin_rpy" value="${M_PI/2} 0.752 -${M_PI/2}" />
-	<xacro:property name="joint_5" value="jaco_joint_5" />
-	<xacro:property name="joint_5_axis_xyz" value="0 0 1" />
-	<xacro:property name="joint_5_origin_xyz" value="0.0343 0 -0.06588" />
-	<xacro:property name="joint_5_origin_rpy" value="0.959 -0.045 -1.539" />
-	<xacro:property name="joint_6" value="jaco_joint_6" />
-	<xacro:property name="joint_6_axis_xyz" value="0 0 1" />
-	<xacro:property name="joint_6_origin_xyz" value="0.0343 0 -0.06588" />
-	<xacro:property name="joint_6_origin_rpy" value="0.953 0.139 -1.669" />
-	<xacro:property name="joint_finger_1" value="jaco_joint_finger_1" />
-	<xacro:property name="joint_finger_1_axis_xyz" value="0 0 1" />
-	<xacro:property name="joint_finger_1_origin_xyz" value="-0.032578 0.0033 -0.12131" />
-	<xacro:property name="joint_finger_1_origin_rpy" value="-1.7983 1.117 3.1416" />
-	<xacro:property name="joint_finger_1_lower_limit" value="0" />
-	<xacro:property name="joint_finger_1_upper_limit" value="${M_PI/180*40}" />
-	<xacro:property name="joint_finger_3" value="jaco_joint_finger_3" />
-	<xacro:property name="joint_finger_3_axis_xyz" value="0 0 1" />
-	<xacro:property name="joint_finger_3_origin_xyz" value="0.027788 -0.0206 -0.12131" />
-	<xacro:property name="joint_finger_3_origin_rpy" value="-1.6222 1.117 -0.23615" />
-	<xacro:property name="joint_finger_3_lower_limit" value="0" />
-	<xacro:property name="joint_finger_3_upper_limit" value="${M_PI/180*40}" />
-	<xacro:property name="joint_finger_2" value="jaco_joint_finger_2" />
-	<xacro:property name="joint_finger_2_axis_xyz" value="0 0 1" />
-	<xacro:property name="joint_finger_2_origin_xyz" value="0.027788 0.0206 -0.12131" />
-	<xacro:property name="joint_finger_2_origin_rpy" value="-1.5161 1.1459 0.23978" />
-	<xacro:property name="joint_finger_2_lower_limit" value="0" />
-	<xacro:property name="joint_finger_2_upper_limit" value="${M_PI/180*40}" />
-	<xacro:property name="joint_finger_tip_1" value="jaco_joint_finger_tip_1" />
-	<xacro:property name="joint_finger_tip_1_axis_xyz" value="0 0 1" />
-	<xacro:property name="joint_finger_tip_1_origin_xyz" value="0.044094 -0.0029 0" />
-	<xacro:property name="joint_finger_tip_1_origin_rpy" value="0 0 0" />
-	<xacro:property name="joint_finger_tip_1_lower_limit" value="0" />
-	<xacro:property name="joint_finger_tip_1_upper_limit" value="${M_PI/180*40}" />
-	<xacro:property name="joint_finger_tip_2" value="jaco_joint_finger_tip_2" />
-	<xacro:property name="joint_finger_tip_2_axis_xyz" value="0 0 1" />
-	<xacro:property name="joint_finger_tip_2_origin_xyz" value="0.044094 -0.0029 0" />
-	<xacro:property name="joint_finger_tip_2_origin_rpy" value="0 0 0" />
-	<xacro:property name="joint_finger_tip_2_lower_limit" value="0" />
-	<xacro:property name="joint_finger_tip_2_upper_limit" value="${M_PI/180*40}" />
-	<xacro:property name="joint_finger_tip_3" value="jaco_joint_finger_tip_3" />
-	<xacro:property name="joint_finger_tip_3_axis_xyz" value="0 0 1" />
-	<xacro:property name="joint_finger_tip_3_origin_xyz" value="0.044094 -0.0029 0" />
-	<xacro:property name="joint_finger_tip_3_origin_rpy" value="0 0 0" />
-	<xacro:property name="joint_finger_tip_3_lower_limit" value="0" />
-	<xacro:property name="joint_finger_tip_3_upper_limit" value="${M_PI/180*40}" />
+  <xacro:property name="joint_1_axis_xyz" value="0 0 1" />
+  <xacro:property name="joint_1_origin_xyz" value="0 0 0.1535" />
+  <xacro:property name="joint_1_origin_rpy" value="${M_PI} 0 0" />
+  <xacro:property name="joint_2" value="jaco_joint_2" />
+  <xacro:property name="joint_2_axis_xyz" value="0 0 1" />
+  <xacro:property name="joint_2_origin_xyz" value="0 0 -0.1185" />
+  <xacro:property name="joint_2_origin_rpy" value="-${M_PI/2} -${M_PI/2} 0" />
+  <xacro:property name="joint_3" value="jaco_joint_3" />
+  <xacro:property name="joint_3_axis_xyz" value="0 0 1" />
+  <xacro:property name="joint_3_origin_xyz" value="0.41 0 0" />
+  <xacro:property name="joint_3_origin_rpy" value="${M_PI} 0 ${M_PI}" />
+  <xacro:property name="joint_4" value="jaco_joint_4" />
+  <xacro:property name="joint_4_axis_xyz" value="0 0 1" />
+  <xacro:property name="joint_4_origin_xyz" value="0.207 0 -0.01125" />
+  <xacro:property name="joint_4_origin_rpy" value="0 -${M_PI/2} 0" />
+  <xacro:property name="joint_5" value="jaco_joint_5" />
+  <xacro:property name="joint_5_axis_xyz" value="0 0 1" />
+  <xacro:property name="joint_5_origin_xyz" value="0.0343 0 -0.06588" />
+  <xacro:property name="joint_5_origin_rpy" value="0 ${M_PI/180*55} ${M_PI}" />
+  <xacro:property name="joint_6" value="jaco_joint_6" />
+  <xacro:property name="joint_6_axis_xyz" value="0 0 1" />
+  <xacro:property name="joint_6_origin_xyz" value="0.0343 0 -0.06588" />
+  <xacro:property name="joint_6_origin_rpy" value="0 ${M_PI/180*55} ${M_PI}" />
+  <xacro:property name="joint_finger_1" value="jaco_joint_finger_1" />
+  <xacro:property name="joint_finger_1_axis_xyz" value="0 0 1" />
+  <xacro:property name="joint_finger_1_origin_xyz" value="-0.032578 0.0033 -0.12131" />
+  <xacro:property name="joint_finger_1_origin_rpy" value="-1.7983 1.117 3.1416" />
+  <xacro:property name="joint_finger_1_lower_limit" value="0" />
+  <xacro:property name="joint_finger_1_upper_limit" value="${M_PI/180*40}" />
+  <xacro:property name="joint_finger_3" value="jaco_joint_finger_3" />
+  <xacro:property name="joint_finger_3_axis_xyz" value="0 0 1" />
+  <xacro:property name="joint_finger_3_origin_xyz" value="0.027788 -0.0206 -0.12131" />
+  <xacro:property name="joint_finger_3_origin_rpy" value="-1.6222 1.117 -0.23615" />
+  <xacro:property name="joint_finger_3_lower_limit" value="0" />
+  <xacro:property name="joint_finger_3_upper_limit" value="${M_PI/180*40}" />
+  <xacro:property name="joint_finger_2" value="jaco_joint_finger_2" />
+  <xacro:property name="joint_finger_2_axis_xyz" value="0 0 1" />
+  <xacro:property name="joint_finger_2_origin_xyz" value="0.027788 0.0206 -0.12131" />
+  <xacro:property name="joint_finger_2_origin_rpy" value="-1.5161 1.1459 0.23978" />
+  <xacro:property name="joint_finger_2_lower_limit" value="0" />
+  <xacro:property name="joint_finger_2_upper_limit" value="${M_PI/180*40}" />
+  <xacro:property name="joint_finger_tip_1" value="jaco_joint_finger_tip_1" />
+  <xacro:property name="joint_finger_tip_1_axis_xyz" value="0 0 1" />
+  <xacro:property name="joint_finger_tip_1_origin_xyz" value="0.044094 -0.0029 0" />
+  <xacro:property name="joint_finger_tip_1_origin_rpy" value="0 0 0" />
+  <xacro:property name="joint_finger_tip_1_lower_limit" value="0" />
+  <xacro:property name="joint_finger_tip_1_upper_limit" value="${M_PI/180*40}" />
+  <xacro:property name="joint_finger_tip_2" value="jaco_joint_finger_tip_2" />
+  <xacro:property name="joint_finger_tip_2_axis_xyz" value="0 0 1" />
+  <xacro:property name="joint_finger_tip_2_origin_xyz" value="0.044094 -0.0029 0" />
+  <xacro:property name="joint_finger_tip_2_origin_rpy" value="0 0 0" />
+  <xacro:property name="joint_finger_tip_2_lower_limit" value="0" />
+  <xacro:property name="joint_finger_tip_2_upper_limit" value="${M_PI/180*40}" />
+  <xacro:property name="joint_finger_tip_3" value="jaco_joint_finger_tip_3" />
+  <xacro:property name="joint_finger_tip_3_axis_xyz" value="0 0 1" />
+  <xacro:property name="joint_finger_tip_3_origin_xyz" value="0.044094 -0.0029 0" />
+  <xacro:property name="joint_finger_tip_3_origin_rpy" value="0 0 0" />
+  <xacro:property name="joint_finger_tip_3_lower_limit" value="0" />
+  <xacro:property name="joint_finger_tip_3_upper_limit" value="${M_PI/180*40}" />
 	<xacro:macro name="jaco_link" params="link_name">
 		<link name="${link_name}">
