Commit message: Added an option to use a primitive-shape--based collision model.
This model is much better for collision detection, raycasting and other geometrical computations.

The model is only approximate.

File: jaco_description/robots/cylinder_arm.urdf.xacro (robot description, xacro)
@@ -13,4 +13,5 @@
 	xmlns:physics="http://playerstage.sourceforge.net/gazebo/xmlschema/#physics"
 	xmlns:xacro="http://ros.org/wiki/xacro" name="jaco">
+	<xacro:arg name="simple_collisions" default="0" />
 	<xacro:include filename="$(find jaco_description)/urdf/jaco_arm.urdf.xacro" />
 	<link name="root">
@@ -70,4 +71,4 @@
 	  <child link="support" />
 	</joint>
-	<xacro:jaco_arm parent="support" xyz="0 0 0.2" rpy="0 0 0" />
+	<xacro:jaco_arm parent="support" xyz="0 0 0.2" rpy="0 0 0" simple_collisions="$(arg simple_collisions)" />
 </robot>

File: jaco_description/robots/standalone_arm.urdf.xacro (robot description, xacro)
@@ -13,4 +13,5 @@
 	xmlns:physics="http://playerstage.sourceforge.net/gazebo/xmlschema/#physics"
 	xmlns:xacro="http://ros.org/wiki/xacro" name="jaco">
+	<xacro:arg name="simple_collisions" default="0" />
 	<xacro:include filename="$(find jaco_description)/urdf/jaco_arm.urdf.xacro" />
 	<link name="root">
@@ -28,4 +29,4 @@
 		</collision>
 	</link>
-	<xacro:jaco_arm parent="root" xyz="0 0 0" rpy="0 0 0" />
+	<xacro:jaco_arm parent="root" xyz="0 0 0" rpy="0 0 0" simple_collisions="$(arg simple_collisions)" />
 </robot>

File: jaco_description/urdf/jaco_arm.urdf.xacro (robot description, xacro)
@@ -86,8 +86,265 @@
   <xacro:property name="joint_finger_tip_3_lower_limit" value="0" />
   <xacro:property name="joint_finger_tip_3_upper_limit" value="${M_PI/180*40}" />
-	<xacro:macro name="jaco_link" params="link_name">
-		<link name="${link_name}">
+  <!-- Simple collision elements for all links. -->
+  <xacro:property name="link_base_link_data">
+      <link_data>
+          <collision>
+            <origin rpy="0 0 0" xyz="0 0 0.076" />
+            <geometry>
+                <cylinder length="0.154" radius="0.043" />
+            </geometry>
+        </collision>
+        <collision>
+            <origin rpy="0 0 0" xyz="0 0.02 0.097" />
+            <geometry>
+                <box size="0.08 0.05 0.052" />
+            </geometry>
+        </collision>
+      </link_data>
+  </xacro:property>
+  <xacro:property name="link_1_link_data">
+      <link_data>
+            <collision>
+                <origin rpy="0 0 0" xyz="0 0 -0.02" />
+                <geometry>
+                    <cylinder length="0.04" radius="0.043" />
+                </geometry>
+            </collision>
+            <collision>
+                <origin rpy="${M_PI/2.0} 0 0" xyz="0 ${0.0395/2} -0.11925" />
+                <geometry>
+                    <cylinder length="0.045" radius="0.043" />
+                </geometry>
+            </collision>
+            <collision>
+                <origin rpy="${M_PI/2.0} 0 0" xyz="0 ${0.0395/2+0.024} -0.11925" />
+                <geometry>
+                    <cylinder length="0.004" radius="0.02" />
+                </geometry>
+            </collision>
+            <collision>
+                <origin rpy="0.06 0 0" xyz="0 0.031 -0.07875" />
+                <geometry>
+                    <box size="0.079 0.027 0.080" />
+                </geometry>
+	     </collision>
+	     <collision>
+                <origin rpy="-0.7 0 0" xyz="0 0 -0.044" />
+                <geometry>
+                    <cylinder length="0.035" radius="0.045" />
+                </geometry>
+            </collision>
+      </link_data>
+  </xacro:property>
+  <xacro:property name="link_2_link_data">
+      <link_data>
+            <collision>
+                <origin rpy="0 0 0" xyz="0 0 -0.022" />
+                <geometry>
+                    <cylinder length="0.042" radius="0.043" />
+                </geometry>
+            </collision>
+            <collision>
+                <origin rpy="0 0 0" xyz="0.411 0 -0.022" />
+                <geometry>
+                    <cylinder length="0.042" radius="0.043" />
+                </geometry>
+            </collision>
+            <collision>
+                <origin rpy="0 0 0" xyz="${0.411/2} 0 -0.022" />
+                <geometry>
+                    <box size="0.411 0.082 0.04" />
+                </geometry>
+            </collision>
+        </link_data>
+  </xacro:property>
+  <xacro:property name="link_3_link_data">
+      <link_data>
+            <collision>
+                <origin rpy="0 0 0" xyz="0 0 -0.0225" />
+                <geometry>
+                    <cylinder length="0.045" radius="0.043" />
+                </geometry>
+            </collision>
+            <collision>
+                <origin rpy="0 ${M_PI/2.0} 0" xyz="0.187 0 -0.012" />
+                <geometry>
+                    <cylinder length="0.04" radius="0.034" />
+                </geometry>
+            </collision>
+            <collision>
+                <origin rpy="0 -0.02 0" xyz="${0.25/2-0.02} 0 -0.040" />
+                <geometry>
+                    <box size="0.2 0.03 0.01" />
+                </geometry>
+            </collision>
+            <collision>
+                <origin rpy="0 -0.025 0" xyz="${0.25/2-0.02} 0 -0.035" />
+                <geometry>
+                    <box size="0.2 0.053 0.01" />
+                </geometry>
+            </collision>
+            <collision>
+                <origin rpy="0 -0.05 0" xyz="${0.25/2-0.02} 0 -0.025" />
+                <geometry>
+                    <box size="0.2 0.066 0.02" />
+                </geometry>
+            </collision>
+            <collision>
+                <origin rpy="0 -0.07 0" xyz="${0.25/2-0.02} 0 -0.025" />
+                <geometry>
+                    <box size="0.2 0.066 0.02" />
+                </geometry>
+            </collision>
+            <collision>
+                <origin rpy="0 -0.20 0" xyz="${0.25/2-0.02} 0 -0.013" />
+                <geometry>
+                    <box size="0.18 0.05 0.018" />
+                </geometry>
+            </collision>
+            <collision>
+                <origin rpy="0 -0.26 0" xyz="${0.25/2-0.02} 0 -0.009" />
+                <geometry>
+                    <box size="0.18 0.03 0.016" />
+                </geometry>
+            </collision>
+            <collision>
+                <origin rpy="0 -0.18 0" xyz="0.07 0 -0.025" />
+                <geometry>
+                    <box size="0.13 0.084 0.02" />
+                </geometry>
+            </collision>
+            <collision>
+                <origin rpy="0 -0.18 0" xyz="0.09 0 -0.025" />
+                <geometry>
+                    <box size="0.15 0.072 0.02" />
+                </geometry>
+            </collision>
+        </link_data>
+  </xacro:property>
+  <xacro:property name="link_4_5_link_data">
+      <link_data>
+            <collision>
+                <origin rpy="0 0 0" xyz="0 0 -${0.045/2}" />
+                <geometry>
+                    <cylinder length="0.045" radius="0.034" />
+                </geometry>
+            </collision>
+            <collision>
+                <origin rpy="0 ${-M_PI/8-0.08} 0" xyz="0.008 0 ${-0.03-0.045/4}" />
+                <geometry>
+                    <cylinder length="0.030" radius="0.036" />
+                </geometry>
+            </collision>
+            <collision>
+                <origin rpy="0 ${-M_PI/4-0.16} 0" xyz="0.017 0 ${-0.03-0.045/2}" />
+                <geometry>
+                    <cylinder length="0.045" radius="0.034" />
+                </geometry>
+            </collision>
+        </link_data>
+  </xacro:property>
+  <xacro:property name="link_hand_link_data">
+      <link_data>
+            <collision>
+                <origin rpy="0 0 0" xyz="0 0 -${0.035/2}" />
+                <geometry>
+                    <cylinder length="0.035" radius="0.034" />
+                </geometry>
+            </collision>
+            <collision>
+                <origin rpy="-0.05 0.45 0" xyz="-0.022 0 -0.06" />
+                <geometry>
+                    <cylinder length="0.09" radius="0.035" />
+                </geometry>
+            </collision>
+            <collision>
+                <origin rpy="-0.05 0.45 0" xyz="-0.022 0 -0.06" />
+                <geometry>
+                    <cylinder length="0.11" radius="0.02" />
+                </geometry>
+            </collision>
+            <collision>
+                <origin rpy="-0.25 -0.45 0" xyz="0.018 -0.014 -0.06" />
+                <geometry>
+                    <cylinder length="0.09" radius="0.034" />
+                </geometry>
+            </collision>
+            <collision>
+                <origin rpy="-0.25 -0.45 0" xyz="0.018 -0.014 -0.06" />
+                <geometry>
+                    <cylinder length="0.11" radius="0.02" />
+                </geometry>
+            </collision>
+            <collision>
+                <origin rpy="0.25 -0.45 0" xyz="0.018 0.014 -0.06" />
+                <geometry>
+                    <cylinder length="0.09" radius="0.034" />
+                </geometry>
+            </collision>
+            <collision>
+                <origin rpy="0.25 -0.45 0" xyz="0.018 0.014 -0.06" />
+                <geometry>
+                    <cylinder length="0.11" radius="0.02" />
+                </geometry>
+            </collision>
+            <collision>
+                <origin rpy="0 -0.45 0" xyz="0.052 0 -0.055" />
+                <geometry>
+                    <box size="0.01 0.03 0.07" />
+                </geometry>
+            </collision>
+            <collision>
+                <origin rpy="0 ${M_PI/2.0-0.0} -0.03" xyz="-0.005 0 -0.065" />
+                <geometry>
+                    <cylinder length="0.032" radius="0.05" />
+                </geometry>
+            </collision>
+        </link_data>
+  </xacro:property>
+  <xacro:property name="finger_link_data">
+      <link_data>
+          <collision>
+              <origin rpy="0 0 0" xyz="${0.055/2-0.007} -0.01 0" />
+              <geometry>
+                  <box size="0.055 0.026 0.024" />
+              </geometry>
+          </collision>
+      </link_data>
+  </xacro:property>
+  <xacro:property name="finger_tip_link_data">
+      <link_data>
+          <collision>
+              <origin rpy="0 0 0" xyz="${0.045/2} -0.005 0" />
+              <geometry>
+                  <box size="0.045 0.020 0.024" />
+              </geometry>
+          </collision>
+      </link_data>
+  </xacro:property>
+  <xacro:property name="large_ring_data">
+      <link_data>
+          <collision>
+              <origin rpy="0 0 0" xyz="0 0 0" />
+              <geometry>
+                  <cylinder length="0.023" radius="0.046" />
+              </geometry>
+          </collision>
+      </link_data>
+  </xacro:property>
+   <xacro:property name="small_ring_data">
+      <link_data>
+          <collision>
+              <origin rpy="0 0 0" xyz="0 0 0" />
+              <geometry>
+                  <cylinder length="0.023" radius="0.037" />
+              </geometry>
+          </collision>
+      </link_data>
+  </xacro:property>
+	  <xacro:macro name="jaco_link_with_collisions" params="link_name mass:=1.0 suffix:='' suffix_separator:='' file_suffix:='' simple_collisions:=0 **simple_collision_data">
+	    <link name="${link_name}${suffix_separator}${suffix}">
             <inertial>
-                <mass value="1"/>
+		<mass value="${mass}"/>
                 <inertia ixx="0.1" ixy="0" ixz="0" iyy="0.1" iyz="0" izz="0.1"/>
                 <origin/>
@@ -95,5 +352,5 @@
 			<visual>
 				<geometry>
-					<mesh scale="${M_SCALE} ${M_SCALE} ${M_SCALE}" filename="package://jaco_description/meshes/${link_name}.min.dae" />
+					<mesh scale="${M_SCALE} ${M_SCALE} ${M_SCALE}" filename="package://jaco_description/meshes/${link_name}${file_suffix}.min.dae" />
 				</geometry>
 				<material name="carbon_fiber">
@@ -101,76 +358,36 @@
 				</material>
 			</visual>
+			<xacro:unless value="${simple_collisions}">
 			<collision>
 				<geometry>
-					<mesh scale="${M_SCALE} ${M_SCALE} ${M_SCALE}" filename="package://jaco_description/meshes/${link_name}.stl" />
+					<mesh scale="${M_SCALE} ${M_SCALE} ${M_SCALE}" filename="package://jaco_description/meshes/${link_name}${file_suffix}.stl" />
 				</geometry>
 			</collision>
+			</xacro:unless>
+			<xacro:if value="${simple_collisions}">
+				<xacro:insert_block name="simple_collision_data" />
+			</xacro:if>
 		</link>
 	</xacro:macro>
+	<!-- Backwards compatibility macro for calling without collisions specifications. -->
+	<xacro:macro name="jaco_link" params="link_name">
+		<xacro:jaco_link_with_collisions link_name="${link_name}" simple_collisions="0">
+			  <link_data/>
+		</xacro:jaco_link_with_collisions>
+	</xacro:macro>
 	<xacro:macro name="jaco_link_suffix" params="link_name suffix">
-		<link name="${link_name}_${suffix}">
-            <inertial>
-                <mass value="0.25"/>
-                <inertia ixx="0.01" ixy="0" ixz="0" iyy="0.01" iyz="0" izz="0.01"/>
-                <origin/>
-            </inertial>
-			<visual>
-				<geometry>
-					<mesh scale="${M_SCALE} ${M_SCALE} ${M_SCALE}" filename="package://jaco_description/meshes/${link_name}.min.dae" />
-				</geometry>
-				<material name="carbon_fiber">
-					<color rgba="0.792156862745098 0.819607843137255 0.933333333333333 1" />
-				</material>
-			</visual>
-			<collision>
-				<geometry>
-					<mesh scale="${M_SCALE} ${M_SCALE} ${M_SCALE}" filename="package://jaco_description/meshes/${link_name}.stl" />
-				</geometry>
-			</collision>
-		</link>
+		<xacro:jaco_link_with_collisions mass="0.25" link_name="${link_name}" suffix="${suffix}" suffix_separator="_">
+			<link_data/>
+		</xacro:jaco_link_with_collisions>
 	</xacro:macro>
 	<xacro:macro name="jaco_link_4_5" params="link_name suffix">
-		<link name="${link_name}_${suffix}">
-            <inertial>
-                <mass value="0.5"/>
-                <inertia ixx="0.01" ixy="0" ixz="0" iyy="0.01" iyz="0" izz="0.01"/>
-                <origin/>
-            </inertial>
-			<visual>
-				<geometry>
-					<mesh scale="${M_SCALE} ${M_SCALE} ${M_SCALE}" filename="package://jaco_description/meshes/${link_name}_4_5.min.dae" />
-				</geometry>
-				<material name="carbon_fiber">
-					<color rgba="0.792156862745098 0.819607843137255 0.933333333333333 1" />
-				</material>
-			</visual>
-			<collision>
-				<geometry>
-					<mesh scale="${M_SCALE} ${M_SCALE} ${M_SCALE}" filename="package://jaco_description/meshes/${link_name}_4_5.stl" />
-				</geometry>
-			</collision>
-		</link>
+		<xacro:jaco_link_with_collisions mass="0.5" link_name="${link_name}" suffix="${suffix}" suffix_separator="_" file_suffix="_4_5">
+			<link_data/>
+		</xacro:jaco_link_with_collisions>
 	</xacro:macro>
 	<xacro:macro name="jaco_ring_cover" params="suffix size">
-		<link name="jaco_${size}_ring_cover_${suffix}">
-            <inertial>
-                <mass value="0"/>
-                <inertia ixx="0" ixy="0" ixz="0" iyy="0" iyz="0" izz="0"/>
-                <origin/>
-            </inertial>
-			<visual>
-				<geometry>
-					<mesh scale="${M_SCALE} ${M_SCALE} ${M_SCALE}" filename="package://jaco_description/meshes/jaco_${size}_ring_cover.min.dae" />
-				</geometry>
-				<material name="carbon_fiber">
-					<color rgba="0.792156862745098 0.819607843137255 0.933333333333333 1" />
-				</material>
-			</visual>
-			<collision>
-				<geometry>
-					<mesh scale="${M_SCALE} ${M_SCALE} ${M_SCALE}" filename="package://jaco_description/meshes/jaco_${size}_ring_cover.stl" />
-				</geometry>
-			</collision>
-		</link>
+		<xacro:jaco_link_with_collisions mass="0.001" link_name="jaco_${size}_ring_cover" suffix="${suffix}" suffix_separator="_">
+			<link_data/>
+		</xacro:jaco_link_with_collisions>
 	</xacro:macro>
 	<xacro:macro name="jaco_joint" params="joint_name type parent child joint_axis_xyz joint_origin_xyz joint_origin_rpy lower_limit upper_limit">
@@ -203,59 +420,59 @@
         </transmission>
 	</xacro:macro>
-	<xacro:macro name="jaco_arm" params="parent xyz rpy">
+	<xacro:macro name="jaco_arm" params="parent xyz rpy simple_collisions:=0 gazebo_robot_name:=robot_description">
         <gazebo>
             <plugin filename="libgazebo_ros_control.so" name="gazebo_ros_controller_manager">
                 <!-- <robotNamespace>/</robotNamespace> -->
-                <robotParam>robot_description</robotParam>
+		<robotParam>${gazebo_robot_name}</robotParam>
             </plugin>
         </gazebo>
-		<xacro:jaco_link link_name="${link_base}" />
+		<xacro:jaco_link_with_collisions link_name="${link_base}" simple_collisions="${simple_collisions}"><xacro:insert_block name="link_base_link_data" /></xacro:jaco_link_with_collisions>
 		<xacro:jaco_joint joint_name="${joint_base}" type="fixed" parent="${parent}" child="${link_base}" joint_axis_xyz="${joint_base_axis_xyz}" joint_origin_xyz="${xyz}" joint_origin_rpy="${rpy}" lower_limit="-${J_LIM}" upper_limit="${J_LIM}" />
-		<xacro:jaco_link link_name="${link_1}" />
+		<xacro:jaco_link_with_collisions link_name="${link_1}" simple_collisions="${simple_collisions}"><xacro:insert_block name="link_1_link_data" /></xacro:jaco_link_with_collisions>
 		<xacro:jaco_joint joint_name="${joint_1}" type="revolute" parent="${link_base}" child="${link_1}" joint_axis_xyz="${joint_1_axis_xyz}" joint_origin_xyz="${joint_1_origin_xyz}" joint_origin_rpy="${joint_1_origin_rpy}" lower_limit="-${J_LIM}" upper_limit="${J_LIM}" />
         <xacro:jaco_transmission joint_name="${joint_1}" />
-		<xacro:jaco_link link_name="${link_2}" />
+		<xacro:jaco_link_with_collisions link_name="${link_2}" simple_collisions="${simple_collisions}"><xacro:insert_block name="link_2_link_data" /></xacro:jaco_link_with_collisions>
 		<xacro:jaco_joint joint_name="${joint_2}" type="revolute" parent="${link_1}" child="${link_2}" joint_axis_xyz="${joint_2_axis_xyz}" joint_origin_xyz="${joint_2_origin_xyz}" joint_origin_rpy="${joint_2_origin_rpy}" lower_limit="0" upper_limit="${J_LIM}" />
         <xacro:jaco_transmission joint_name="${joint_2}" />
-		<xacro:jaco_link link_name="${link_3}" />
+		<xacro:jaco_link_with_collisions link_name="${link_3}" simple_collisions="${simple_collisions}"><xacro:insert_block name="link_3_link_data" /></xacro:jaco_link_with_collisions>
 		<xacro:jaco_joint joint_name="${joint_3}" type="revolute" parent="${link_2}" child="${link_3}" joint_axis_xyz="${joint_3_axis_xyz}" joint_origin_xyz="${joint_3_origin_xyz}" joint_origin_rpy="${joint_3_origin_rpy}" lower_limit="0" upper_limit="${J_LIM}" />
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