Commit message: mico description adaptions

File: mico_description/robots/standalone_arm.urdf (robot description, URDF)
Before this commit: robot jaco, 14 links, 13 joints
Links:
- removed link jaco_large_ring_cover_1
- removed link jaco_large_ring_cover_2
- removed link jaco_large_ring_cover_3
- removed link jaco_link_1
- removed link jaco_link_2
- removed link jaco_link_3
- removed link jaco_link_4
- removed link jaco_link_5
- removed link jaco_link_base
- removed link jaco_link_hand
- removed link jaco_small_ring_cover_1
- removed link jaco_small_ring_cover_2
- removed link jaco_small_ring_cover_3
- added link mico_large_ring_cover_1; collision mesh filename=package://mico_description/meshes/mico_large_ring_cover.dae scale=0.0254 0.0254 0.0254; visual mesh filename=package://mico_description/meshes/mico_large_ring_cover.dae scale=0.0254 0.0254 0.0254
- added link mico_large_ring_cover_2; collision mesh filename=package://mico_description/meshes/mico_large_ring_cover.dae scale=0.0254 0.0254 0.0254; visual mesh filename=package://mico_description/meshes/mico_large_ring_cover.dae scale=0.0254 0.0254 0.0254
- added link mico_large_ring_cover_3; collision mesh filename=package://mico_description/meshes/mico_large_ring_cover.dae scale=0.0254 0.0254 0.0254; visual mesh filename=package://mico_description/meshes/mico_large_ring_cover.dae scale=0.0254 0.0254 0.0254
- added link mico_link_1; collision mesh filename=package://mico_description/meshes/mico_link_1.dae scale=1.0000 1.0000 1.0000; visual mesh filename=package://mico_description/meshes/mico_link_1.dae scale=1.0000 1.0000 1.0000
- added link mico_link_2; collision mesh filename=package://mico_description/meshes/mico_link_2.dae scale=1.0000 1.0000 1.0000; visual mesh filename=package://mico_description/meshes/mico_link_2.dae scale=1.0000 1.0000 1.0000
- added link mico_link_3; collision mesh filename=package://mico_description/meshes/mico_link_3.dae scale=1.0000 1.0000 1.0000; visual mesh filename=package://mico_description/meshes/mico_link_3.dae scale=1.0000 1.0000 1.0000
- added link mico_link_4; collision mesh filename=package://mico_description/meshes/mico_link_4_5.dae scale=1.0000 1.0000 1.0000; visual mesh filename=package://mico_description/meshes/mico_link_4_5.dae scale=1.0000 1.0000 1.0000
- added link mico_link_5; collision mesh filename=package://mico_description/meshes/mico_link_4_5.dae scale=1.0000 1.0000 1.0000; visual mesh filename=package://mico_description/meshes/mico_link_4_5.dae scale=1.0000 1.0000 1.0000
- added link mico_link_base; collision mesh filename=package://mico_description/meshes/mico_link_base.dae scale=1.0000 1.0000 1.0000; visual mesh filename=package://mico_description/meshes/mico_link_base.dae scale=1.0000 1.0000 1.0000
- added link mico_link_finger_1; collision mesh filename=package://mico_description/meshes/mico_link_finger.dae scale=0.0254 0.0254 0.0254; visual mesh filename=package://mico_description/meshes/mico_link_finger.dae scale=0.0254 0.0254 0.0254
- added link mico_link_finger_2; collision mesh filename=package://mico_description/meshes/mico_link_finger.dae scale=0.0254 0.0254 0.0254; visual mesh filename=package://mico_description/meshes/mico_link_finger.dae scale=0.0254 0.0254 0.0254
- added link mico_link_finger_tip_1; collision mesh filename=package://mico_description/meshes/mico_link_finger_tip.dae scale=0.0254 0.0254 0.0254; visual mesh filename=package://mico_description/meshes/mico_link_finger_tip.dae scale=0.0254 0.0254 0.0254
- added link mico_link_finger_tip_2; collision mesh filename=package://mico_description/meshes/mico_link_finger_tip.dae scale=0.0254 0.0254 0.0254; visual mesh filename=package://mico_description/meshes/mico_link_finger_tip.dae scale=0.0254 0.0254 0.0254
- added link mico_link_hand; collision mesh filename=package://mico_description/meshes/mico_link_hand.dae scale=1.0000 1.0000 1.0000; visual mesh filename=package://mico_description/meshes/mico_link_hand.dae scale=1.0000 1.0000 1.0000
- added link mico_small_ring_cover_1; collision mesh filename=package://mico_description/meshes/mico_small_ring_cover.dae scale=0.0254 0.0254 0.0254; visual mesh filename=package://mico_description/meshes/mico_small_ring_cover.dae scale=0.0254 0.0254 0.0254
- added link mico_small_ring_cover_2; collision mesh filename=package://mico_description/meshes/mico_small_ring_cover.dae scale=0.0254 0.0254 0.0254; visual mesh filename=package://mico_description/meshes/mico_small_ring_cover.dae scale=0.0254 0.0254 0.0254
- added link mico_small_ring_cover_3; collision mesh filename=package://mico_description/meshes/mico_small_ring_cover.dae scale=0.0254 0.0254 0.0254; visual mesh filename=package://mico_description/meshes/mico_small_ring_cover.dae scale=0.0254 0.0254 0.0254
Joints:
- removed joint jaco_joint_1
- removed joint jaco_joint_2
- removed joint jaco_joint_3
- removed joint jaco_joint_4
- removed joint jaco_joint_5
- removed joint jaco_joint_6
- removed joint jaco_joint_base
- removed joint jaco_large_ring_cover_1_joint
- removed joint jaco_large_ring_cover_2_joint
- removed joint jaco_large_ring_cover_3_joint
- removed joint jaco_large_ring_cover_4_joint
- removed joint jaco_large_ring_cover_5_joint
- removed joint jaco_large_ring_cover_6_joint
- added joint mico_joint_1: type continuous, parent mico_link_base, child mico_link_1, origin xyz=0 0 0.1535 rpy=3.14159265359 0 0, axis 0 0 1, limit lower=-6.28318530718 upper=6.28318530718 effort=30 velocity=5
- added joint mico_joint_2: type revolute, parent mico_link_1, child mico_link_2, origin xyz=0 0 -0.1185 rpy=-1.57079632679 -1.57079632679 0, axis 0 0 1, limit lower=0 upper=6.28318530718 effort=30 velocity=5
- added joint mico_joint_3: type revolute, parent mico_link_2, child mico_link_3, origin xyz=0.41 0 0 rpy=3.14159265359 0 3.14159265359, axis 0 0 1, limit lower=0 upper=6.28318530718 effort=30 velocity=5
- added joint mico_joint_4: type continuous, parent mico_link_3, child mico_link_4, origin xyz=0.207 0 -0.01125 rpy=0 -1.57079632679 0, axis 0 0 1, limit lower=-6.28318530718 upper=6.28318530718 effort=30 velocity=5
- added joint mico_joint_5: type continuous, parent mico_link_4, child mico_link_5, origin xyz=0.0343 0 -0.06588 rpy=0 0.959931088597 3.14159265359, axis 0 0 1, limit lower=-6.28318530718 upper=6.28318530718 effort=30 velocity=5
- added joint mico_joint_6: type continuous, parent mico_link_5, child mico_link_hand, origin xyz=0.0343 0 -0.06588 rpy=0 0.959931088597 3.14159265359, axis 0 0 1, limit lower=-6.28318530718 upper=6.28318530718 effort=30 velocity=5
- added joint mico_joint_base: type fixed, parent root, child mico_link_base, origin xyz=0 0 0 rpy=0 0 0, axis 0 0 0, limit lower=-6.28318530718 upper=6.28318530718 effort=30 velocity=5
- added joint mico_joint_finger_1: type revolute, parent mico_link_hand, child mico_link_finger_1, origin xyz=-0.032578 0.0033 -0.12131 rpy=-1.7983 1.117 3.1416, axis 0 0 1, limit lower=0 upper=0.698131700798 effort=30 velocity=5
- added joint mico_joint_finger_2: type revolute, parent mico_link_hand, child mico_link_finger_2, origin xyz=0.027788 0.0206 -0.12131 rpy=-1.5161 1.1459 0.23978, axis 0 0 1, limit lower=0 upper=0.698131700798 effort=30 velocity=5
- added joint mico_joint_finger_tip_1: type revolute, parent mico_link_finger_1, child mico_link_finger_tip_1, origin xyz=0.044094 -0.0029 0 rpy=0 0 0, axis 0 0 1, limit lower=0 upper=0.698131700798 effort=30 velocity=5
- added joint mico_joint_finger_tip_2: type revolute, parent mico_link_finger_2, child mico_link_finger_tip_2, origin xyz=0.044094 -0.0029 0 rpy=0 0 0, axis 0 0 1, limit lower=0 upper=0.698131700798 effort=30 velocity=5
- added joint mico_large_ring_cover_1_joint: type fixed, parent mico_link_base, child mico_large_ring_cover_1, origin xyz=0 0 0.1535 rpy=3.14159265359 0 0, axis 0 0 1, limit lower=-6.28318530718 upper=6.28318530718 effort=30 velocity=5
- added joint mico_large_ring_cover_2_joint: type fixed, parent mico_link_1, child mico_large_ring_cover_2, origin xyz=0 0 -0.1185 rpy=-1.57079632679 -1.57079632679 0, axis 0 0 1, limit lower=0 upper=6.28318530718 effort=30 velocity=5
- added joint mico_large_ring_cover_3_joint: type fixed, parent mico_link_2, child mico_large_ring_cover_3, origin xyz=0.41 0 0 rpy=3.14159265359 0 3.14159265359, axis 0 0 1, limit lower=0 upper=6.28318530718 effort=30 velocity=5
- added joint mico_large_ring_cover_4_joint: type fixed, parent mico_link_3, child mico_small_ring_cover_1, origin xyz=0.207 0 -0.01125 rpy=0 -1.57079632679 0, axis 0 0 1, limit lower=-6.28318530718 upper=6.28318530718 effort=30 velocity=5
- added joint mico_large_ring_cover_5_joint: type fixed, parent mico_link_4, child mico_small_ring_cover_2, origin xyz=0.0343 0 -0.06588 rpy=0 0.959931088597 3.14159265359, axis 0 0 1, limit lower=-6.28318530718 upper=6.28318530718 effort=30 velocity=5
- added joint mico_large_ring_cover_6_joint: type fixed, parent mico_link_5, child mico_small_ring_cover_3, origin xyz=0.0343 0 -0.06588 rpy=0 0.959931088597 3.14159265359, axis 0 0 1, limit lower=-6.28318530718 upper=6.28318530718 effort=30 velocity=5

Commit message: Second positions fix

File: mico_description/robots/standalone_arm.urdf (robot description, URDF)
Before this commit: robot mico, 18 links, 17 joints
Joints:
- joint mico_joint_3: origin xyz=0.41 0 0 rpy=3.14159265359 0 3.14159265359 -> xyz=0.29 0 0 rpy=3.14159265359 0 3.14159265359
- joint mico_joint_4: origin xyz=0.207 0 -0.01125 rpy=0 -1.57079632679 0 -> xyz=0.123 0 -0.01125 rpy=0 -1.57079632679 0
- joint mico_joint_finger_1: origin xyz=-0.032578 0.0033 -0.12131 rpy=-1.7983 1.117 3.1416 -> xyz=-0.03978 0 -0.10071 rpy=-1.7983 1.117 3.1416
- joint mico_joint_finger_2: origin xyz=0.027788 0.0206 -0.12131 rpy=-1.5161 1.1459 0.23978 -> xyz=0.03569 0 -0.10071 rpy=-1.5161 1.1459 0.23978
- joint mico_large_ring_cover_3_joint: origin xyz=0.41 0 0 rpy=3.14159265359 0 3.14159265359 -> xyz=0.29 0 0 rpy=3.14159265359 0 3.14159265359
- joint mico_large_ring_cover_4_joint: origin xyz=0.207 0 -0.01125 rpy=0 -1.57079632679 0 -> xyz=0.123 0 -0.00845 rpy=0 -1.57079632679 0

Commit message: moveitmodel

File: mico_description/robots/standalone_arm.urdf (robot description, URDF)
Before this commit: robot mico, 18 links, 17 joints
Joints:
- joint mico_joint_finger_1: origin xyz=-0.03978 0 -0.10071 rpy=-1.7983 1.117 3.1416 -> xyz=-0.031 0 -0.10071 rpy=-1.5707 0.9666 3.1416
- joint mico_joint_finger_2: origin xyz=0.03569 0 -0.10071 rpy=-1.5161 1.1459 0.23978 -> xyz=0.031 0 -0.10071 rpy=-1.5707 0.9666 0.0

File: mico_description/urdf/mico_arm.urdf.xacro (robot description, xacro)
@@ -53,12 +53,12 @@
   <xacro:property name="joint_finger_1" value="mico_joint_finger_1" />
   <xacro:property name="joint_finger_1_axis_xyz" value="0 0 1" />
-  <xacro:property name="joint_finger_1_origin_xyz" value="-0.03978 0 -0.10071" />
-  <xacro:property name="joint_finger_1_origin_rpy" value="-1.7983 1.117 3.1416" />
+  <xacro:property name="joint_finger_1_origin_xyz" value="-0.031 0 -0.10071" />
+  <xacro:property name="joint_finger_1_origin_rpy" value="-1.5707 1.5707 3.1416" />
   <xacro:property name="joint_finger_1_lower_limit" value="0" />
   <xacro:property name="joint_finger_1_upper_limit" value="${M_PI/180*40}" />
   <xacro:property name="joint_finger_2" value="mico_joint_finger_2" />
   <xacro:property name="joint_finger_2_axis_xyz" value="0 0 1" />
-  <xacro:property name="joint_finger_2_origin_xyz" value="0.03569 0 -0.10071" />
-  <xacro:property name="joint_finger_2_origin_rpy" value="-1.5161 1.1459 0.23978" />
+  <xacro:property name="joint_finger_2_origin_xyz" value="0.031 0 -0.10071" />
+  <xacro:property name="joint_finger_2_origin_rpy" value="-1.5707 1.5707 0.0" />
   <xacro:property name="joint_finger_2_lower_limit" value="0" />
   <xacro:property name="joint_finger_2_upper_limit" value="${M_PI/180*40}" />

Commit message: commented out the fingers

File: mico_description/robots/standalone_arm.urdf (robot description, URDF)
Before this commit: robot mico, 18 links, 17 joints
Links:
- removed link mico_link_finger_1
- removed link mico_link_finger_2
- removed link mico_link_finger_tip_1
- removed link mico_link_finger_tip_2
Joints:
- removed joint mico_joint_finger_1
- removed joint mico_joint_finger_2
- removed joint mico_joint_finger_tip_1
- removed joint mico_joint_finger_tip_2

Commit message: Added first part of the fingers

File: mico_description/robots/standalone_arm.urdf (robot description, URDF)
Before this commit: robot mico, 14 links, 13 joints
Links:
- added link mico_link_finger_1; collision mesh filename=package://mico_description/meshes/mico_link_finger.dae scale=0.0254 0.0254 0.0254; visual mesh filename=package://mico_description/meshes/mico_link_finger.dae scale=0.0254 0.0254 0.0254
- added link mico_link_finger_2; collision mesh filename=package://mico_description/meshes/mico_link_finger.dae scale=0.0254 0.0254 0.0254; visual mesh filename=package://mico_description/meshes/mico_link_finger.dae scale=0.0254 0.0254 0.0254
Joints:
- added joint mico_joint_finger_1: type revolute, parent mico_link_hand, child mico_link_finger_1, origin xyz=-0.03978 0 -0.10071 rpy=-1.5707 0.9666 3.1416, axis 0 0 1, limit lower=0 upper=0.698131700798 effort=30 velocity=5
- added joint mico_joint_finger_2: type revolute, parent mico_link_hand, child mico_link_finger_2, origin xyz=0.03978 0 -0.10071 rpy=-1.5707 0.9666 0.0, axis 0 0 1, limit lower=0 upper=0.698131700798 effort=30 velocity=5

Commit message: Mico description update

File: mico_description/robots/standalone_arm.urdf (robot description, URDF)
Before this commit: robot mico, 16 links, 15 joints
Links:
- added link mico_link_finger_tip_1; collision mesh filename=package://mico_description/meshes/mico_link_finger_tip.dae scale=0.0254 0.0254 0.0254; visual mesh filename=package://mico_description/meshes/mico_link_finger_tip.dae scale=0.0254 0.0254 0.0254
- added link mico_link_finger_tip_2; collision mesh filename=package://mico_description/meshes/mico_link_finger_tip.dae scale=0.0254 0.0254 0.0254; visual mesh filename=package://mico_description/meshes/mico_link_finger_tip.dae scale=0.0254 0.0254 0.0254
Joints:
- added joint mico_joint_finger_tip_1: type fixed, parent mico_link_finger_1, child mico_link_finger_tip_1, origin xyz=0.044094 -0.0029 0.0 rpy=0 0 0, axis 0 0 1, limit lower=0 upper=0.698131700798 effort=30 velocity=5
- added joint mico_joint_finger_tip_2: type fixed, parent mico_link_finger_2, child mico_link_finger_tip_2, origin xyz=0.044094 -0.0029 0.0 rpy=0 0 0, axis 0 0 1, limit lower=0 upper=0.698131700798 effort=30 velocity=5
- joint mico_joint_finger_1: origin xyz=-0.03978 0 -0.10071 rpy=-1.5707 0.9666 3.1416 -> xyz=-0.03978 0 -0.10071 rpy=-1.5707 1.1 3.1416
- joint mico_joint_finger_2: origin xyz=0.03978 0 -0.10071 rpy=-1.5707 0.9666 0.0 -> xyz=0.03978 0 -0.10071 rpy=-1.5707 1.1 0.0
