Commit message: Fixed the positions of the joints

File: mico_description/urdf/mico_arm.urdf.xacro (robot description, xacro)
@@ -37,9 +37,9 @@
   <xacro:property name="joint_3" value="mico_joint_3" />
   <xacro:property name="joint_3_axis_xyz" value="0 0 1" />
-  <xacro:property name="joint_3_origin_xyz" value="0.41 0 0" />
+  <xacro:property name="joint_3_origin_xyz" value="0.29 0 0" />
   <xacro:property name="joint_3_origin_rpy" value="${M_PI} 0 ${M_PI}" />
   <xacro:property name="joint_4" value="mico_joint_4" />
   <xacro:property name="joint_4_axis_xyz" value="0 0 1" />
-  <xacro:property name="joint_4_origin_xyz" value="0.207 0 -0.01125" />
+  <xacro:property name="joint_4_origin_xyz" value="0.123 0 -0.00845" />
   <xacro:property name="joint_4_origin_rpy" value="0 -${M_PI/2} 0" />
   <xacro:property name="joint_5" value="mico_joint_5" />
@@ -53,17 +53,11 @@
   <xacro:property name="joint_finger_1" value="mico_joint_finger_1" />
   <xacro:property name="joint_finger_1_axis_xyz" value="0 0 1" />
-  <xacro:property name="joint_finger_1_origin_xyz" value="-0.032578 0.0033 -0.12131" />
+  <xacro:property name="joint_finger_1_origin_xyz" value="-0.03978 0 -0.10071" />
   <xacro:property name="joint_finger_1_origin_rpy" value="-1.7983 1.117 3.1416" />
   <xacro:property name="joint_finger_1_lower_limit" value="0" />
   <xacro:property name="joint_finger_1_upper_limit" value="${M_PI/180*40}" />
-  <xacro:property name="joint_finger_3" value="mico_joint_finger_3" />
-  <xacro:property name="joint_finger_3_axis_xyz" value="0 0 1" />
-  <xacro:property name="joint_finger_3_origin_xyz" value="0.027788 -0.0206 -0.12131" />
-  <xacro:property name="joint_finger_3_origin_rpy" value="-1.6222 1.117 -0.23615" />
-  <xacro:property name="joint_finger_3_lower_limit" value="0" />
-  <xacro:property name="joint_finger_3_upper_limit" value="${M_PI/180*40}" />
   <xacro:property name="joint_finger_2" value="mico_joint_finger_2" />
   <xacro:property name="joint_finger_2_axis_xyz" value="0 0 1" />
-  <xacro:property name="joint_finger_2_origin_xyz" value="0.027788 0.0206 -0.12131" />
+  <xacro:property name="joint_finger_2_origin_xyz" value="0.03569 0 -0.10071" />
   <xacro:property name="joint_finger_2_origin_rpy" value="-1.5161 1.1459 0.23978" />
   <xacro:property name="joint_finger_2_lower_limit" value="0" />
@@ -81,10 +75,4 @@
   <xacro:property name="joint_finger_tip_2_lower_limit" value="0" />
   <xacro:property name="joint_finger_tip_2_upper_limit" value="${M_PI/180*40}" />
-  <xacro:property name="joint_finger_tip_3" value="mico_joint_finger_tip_3" />
-  <xacro:property name="joint_finger_tip_3_axis_xyz" value="0 0 1" />
-  <xacro:property name="joint_finger_tip_3_origin_xyz" value="0.044094 -0.0029 0" />
-  <xacro:property name="joint_finger_tip_3_origin_rpy" value="0 0 0" />
-  <xacro:property name="joint_finger_tip_3_lower_limit" value="0" />
-  <xacro:property name="joint_finger_tip_3_upper_limit" value="${M_PI/180*40}" />
 	<xacro:macro name="mico_link" params="link_name">
 		<link name="${link_name}">

Commit message: mico model xacro model update

File: mico_description/urdf/mico_arm.urdf.xacro (robot description, xacro)
@@ -53,12 +53,12 @@
   <xacro:property name="joint_finger_1" value="mico_joint_finger_1" />
   <xacro:property name="joint_finger_1_axis_xyz" value="0 0 1" />
-  <xacro:property name="joint_finger_1_origin_xyz" value="-0.031 0 -0.10071" />
-  <xacro:property name="joint_finger_1_origin_rpy" value="-1.5707 1.5707 3.1416" />
+  <xacro:property name="joint_finger_1_origin_xyz" value="-0.03978 0 -0.10071" />
+  <xacro:property name="joint_finger_1_origin_rpy" value="-1.5707 1.1 3.1416" />
   <xacro:property name="joint_finger_1_lower_limit" value="0" />
   <xacro:property name="joint_finger_1_upper_limit" value="${M_PI/180*40}" />
   <xacro:property name="joint_finger_2" value="mico_joint_finger_2" />
   <xacro:property name="joint_finger_2_axis_xyz" value="0 0 1" />
-  <xacro:property name="joint_finger_2_origin_xyz" value="0.031 0 -0.10071" />
-  <xacro:property name="joint_finger_2_origin_rpy" value="-1.5707 1.5707 0.0" />
+  <xacro:property name="joint_finger_2_origin_xyz" value="0.03978 0 -0.10071" />
+  <xacro:property name="joint_finger_2_origin_rpy" value="-1.5707 1.1 0.0" />
   <xacro:property name="joint_finger_2_lower_limit" value="0" />
   <xacro:property name="joint_finger_2_upper_limit" value="${M_PI/180*40}" />
@@ -192,12 +192,8 @@
 		<xacro:mico_link_suffix link_name="${link_finger}" suffix="2"/>
 		<xacro:mico_finger_joint joint_name="${joint_finger_2}" type="revolute" parent="${link_hand}" child="${link_finger}_2" joint_axis_xyz="${joint_finger_2_axis_xyz}" joint_origin_xyz="${joint_finger_2_origin_xyz}" joint_origin_rpy="${joint_finger_2_origin_rpy}" lower_limit="${joint_finger_2_lower_limit}" upper_limit="${joint_finger_2_upper_limit}" />
-		<xacro:mico_link_suffix link_name="${link_finger}" suffix="3"/>
-		<xacro:mico_finger_joint joint_name="${joint_finger_3}" type="revolute" parent="${link_hand}" child="${link_finger}_3" joint_axis_xyz="${joint_finger_3_axis_xyz}" joint_origin_xyz="${joint_finger_3_origin_xyz}" joint_origin_rpy="${joint_finger_3_origin_rpy}" lower_limit="${joint_finger_3_lower_limit}" upper_limit="${joint_finger_3_upper_limit}" />
 		<xacro:mico_link_suffix link_name="${link_finger_tip}" suffix="1"/>
 		<xacro:mico_finger_joint joint_name="${joint_finger_tip_1}" type="revolute" parent="${link_finger}_1" child="${link_finger_tip}_1" joint_axis_xyz="${joint_finger_tip_1_axis_xyz}" joint_origin_xyz="${joint_finger_tip_1_origin_xyz}" joint_origin_rpy="${joint_finger_tip_1_origin_rpy}" lower_limit="${joint_finger_tip_1_lower_limit}" upper_limit="${joint_finger_tip_1_upper_limit}" />
 		<xacro:mico_link_suffix link_name="${link_finger_tip}" suffix="2"/>
 		<xacro:mico_finger_joint joint_name="${joint_finger_tip_2}" type="revolute" parent="${link_finger}_2" child="${link_finger_tip}_2" joint_axis_xyz="${joint_finger_tip_2_axis_xyz}" joint_origin_xyz="${joint_finger_tip_2_origin_xyz}" joint_origin_rpy="${joint_finger_tip_2_origin_rpy}" lower_limit="${joint_finger_tip_2_lower_limit}" upper_limit="${joint_finger_tip_2_upper_limit}" />
-		<xacro:mico_link_suffix link_name="${link_finger_tip}" suffix="3"/>
-		<xacro:mico_finger_joint joint_name="${joint_finger_tip_3}" type="revolute" parent="${link_finger}_3" child="${link_finger_tip}_3" joint_axis_xyz="${joint_finger_tip_3_axis_xyz}" joint_origin_xyz="${joint_finger_tip_3_origin_xyz}" joint_origin_rpy="${joint_finger_tip_3_origin_rpy}" lower_limit="${joint_finger_tip_3_lower_limit}" upper_limit="${joint_finger_tip_3_upper_limit}" />
 	</xacro:macro>
 </robot>

Commit message: xacro updated to be in line with the urdf

File: mico_description/urdf/mico_arm.urdf.xacro (robot description, xacro)
@@ -13,6 +13,5 @@
 	xmlns:physics="http://playerstage.sourceforge.net/gazebo/xmlschema/#physics"
 	xmlns:xacro="http://ros.org/wiki/xacro">
-  <!-- <xacro:property name="M_SCALE" value="0.0254" /> -->
-  <xacro:property name="M_SCALE" value="1.0" />
+  <xacro:property name="M_SCALE" value="0.0254" />
 	<xacro:property name="M_PI" value="3.1415926535897931" />
 	<xacro:property name="J_LIM" value="${2*M_PI}" />
@@ -79,5 +78,5 @@
 			<visual>
 				<geometry>
-					<mesh scale="${M_SCALE} ${M_SCALE} ${M_SCALE}" filename="package://mico_description/meshes/${link_name}.dae" />
+					<mesh filename="package://mico_description/meshes/${link_name}.dae" />
 				</geometry>
 				<material name="carbon_fiber">
@@ -87,5 +86,5 @@
 			<collision>
 				<geometry>
-					<mesh scale="${M_SCALE} ${M_SCALE} ${M_SCALE}" filename="package://mico_description/meshes/${link_name}.dae" />
+					<mesh filename="package://mico_description/meshes/${link_name}.dae" />
 				</geometry>
 			</collision>
@@ -113,5 +112,5 @@
 			<visual>
 				<geometry>
-					<mesh scale="${M_SCALE} ${M_SCALE} ${M_SCALE}" filename="package://mico_description/meshes/${link_name}_4_5.dae" />
+					<mesh filename="package://mico_description/meshes/${link_name}_4_5.dae" />
 				</geometry>
 				<material name="carbon_fiber">
@@ -121,5 +120,5 @@
 			<collision>
 				<geometry>
-					<mesh scale="${M_SCALE} ${M_SCALE} ${M_SCALE}" filename="package://mico_description/meshes/${link_name}_4_5.dae" />
+					<mesh filename="package://mico_description/meshes/${link_name}_4_5.dae" />
 				</geometry>
 			</collision>
@@ -193,7 +192,7 @@
 		<xacro:mico_finger_joint joint_name="${joint_finger_2}" type="revolute" parent="${link_hand}" child="${link_finger}_2" joint_axis_xyz="${joint_finger_2_axis_xyz}" joint_origin_xyz="${joint_finger_2_origin_xyz}" joint_origin_rpy="${joint_finger_2_origin_rpy}" lower_limit="${joint_finger_2_lower_limit}" upper_limit="${joint_finger_2_upper_limit}" />
 		<xacro:mico_link_suffix link_name="${link_finger_tip}" suffix="1"/>
-		<xacro:mico_finger_joint joint_name="${joint_finger_tip_1}" type="revolute" parent="${link_finger}_1" child="${link_finger_tip}_1" joint_axis_xyz="${joint_finger_tip_1_axis_xyz}" joint_origin_xyz="${joint_finger_tip_1_origin_xyz}" joint_origin_rpy="${joint_finger_tip_1_origin_rpy}" lower_limit="${joint_finger_tip_1_lower_limit}" upper_limit="${joint_finger_tip_1_upper_limit}" />
+		<xacro:mico_finger_joint joint_name="${joint_finger_tip_1}" type="fixed" parent="${link_finger}_1" child="${link_finger_tip}_1" joint_axis_xyz="${joint_finger_tip_1_axis_xyz}" joint_origin_xyz="${joint_finger_tip_1_origin_xyz}" joint_origin_rpy="${joint_finger_tip_1_origin_rpy}" lower_limit="${joint_finger_tip_1_lower_limit}" upper_limit="${joint_finger_tip_1_upper_limit}" />
 		<xacro:mico_link_suffix link_name="${link_finger_tip}" suffix="2"/>
-		<xacro:mico_finger_joint joint_name="${joint_finger_tip_2}" type="revolute" parent="${link_finger}_2" child="${link_finger_tip}_2" joint_axis_xyz="${joint_finger_tip_2_axis_xyz}" joint_origin_xyz="${joint_finger_tip_2_origin_xyz}" joint_origin_rpy="${joint_finger_tip_2_origin_rpy}" lower_limit="${joint_finger_tip_2_lower_limit}" upper_limit="${joint_finger_tip_2_upper_limit}" />
+		<xacro:mico_finger_joint joint_name="${joint_finger_tip_2}" type="fixed" parent="${link_finger}_2" child="${link_finger_tip}_2" joint_axis_xyz="${joint_finger_tip_2_axis_xyz}" joint_origin_xyz="${joint_finger_tip_2_origin_xyz}" joint_origin_rpy="${joint_finger_tip_2_origin_rpy}" lower_limit="${joint_finger_tip_2_lower_limit}" upper_limit="${joint_finger_tip_2_upper_limit}" />
 	</xacro:macro>
 </robot>
